Commit message: Upraveny GAZEBO

File: gazebo_scara_v2_with_gripper/scara_v2_description/urdf/scara_v2_with_gripper_urdf.xacro (robot description, xacro)
@@ -22,7 +22,7 @@
             <origin xyz="0 0 0" rpy="0 0 0" />
             <mass value="1" />
-            <inertia ixx="1" ixy="0" ixz="0"
-                    iyy="1" iyz="0"
-                    izz="1" />
+            <inertia ixx="0.01" ixy="0.01" ixz="0.01"
+                    iyy="0.01" iyz="0"
+                    izz="0.01" />
         </inertial>
         <visual>
@@ -44,8 +44,8 @@
         <inertial>
             <origin xyz="0 0 0" rpy="0 0 0" />
-            <mass value="0" />
-            <inertia ixx="1" ixy="0" ixz="0"
-                    iyy="1" iyz="0"
-                    izz="1" />
+            <mass value="1" />
+            <inertia ixx="0.01" ixy="0.01" ixz="0.01"
+                     iyy="0.01" iyz="0.01"
+                     izz="0.01" />
         </inertial>
         <visual>
@@ -74,7 +74,7 @@
             <origin xyz="0 0 0" rpy="0 0 0" />
             <mass value="1" />
-            <inertia ixx="1" ixy="0" ixz="0"
-                    iyy="1" iyz="0"
-                    izz="1" />
+            <inertia ixx="0.01" ixy="0.01" ixz="0.01"
+                     iyy="0.01" iyz="0.01"
+                     izz="0.01" />
         </inertial>
         <visual>
@@ -105,7 +105,7 @@
             <origin xyz="0 0 0" rpy="0 0 0" />
             <mass value="1" />
-            <inertia ixx="1" ixy="0" ixz="0"
-                     iyy="1" iyz="0"
-                     izz="1" />
+            <inertia ixx="0.01" ixy="0.01" ixz="0.01"
+                     iyy="0.01" iyz="0.01"
+                     izz="0.01" />
         </inertial>
         <visual>
@@ -124,9 +124,10 @@
         </collision>
     </link>
-    <joint name="Joint_ScaraBase" type="fixed">
+    <joint name="Joint_ScaraBase" type="revolute">
         <parent link="BaseBox" />
         <child link="ScaraBase" />
         <origin xyz="0.212 0.58 0.141"  rpy="1.5708 0 0" />
         <axis  xyz="1 0 0" />
+        <limit effort="0" lower="0" upper="0" velocity="0"/>
     </joint>
     <link name="ScaraLink1">
@@ -158,5 +159,5 @@
         <origin xyz="0 0.051 0" rpy="0 0 0" />
         <axis xyz="0 1 0" />
-        <limit effort="0" lower="-1.57079" upper="1.57079" velocity="0"/>
+        <limit effort="1000" lower="-1.57079" upper="1.57079" velocity="0"/>
     </joint>
     <link name="ScaraLink2">
@@ -188,101 +189,102 @@
         <origin xyz="0.24972 -0.081 0" rpy="3.14 -1.5708 0" />
         <axis xyz="0 1 0" />
-        <limit effort="0" lower="-2.65" upper="2.65" velocity="0"/>
+        <limit effort="1000" lower="-2.65" upper="2.65" velocity="0"/>
     </joint>
     <!--**********************************-->
     <!--     GRIPPER JOINTS DEFINITION    -->
-    <link name="GripperBase">
-        <inertial>
-            <origin xyz="0 0 0" rpy="0 0 0" />
-            <mass  value="1" />
-            <inertia  ixx="1E-6" ixy="0" ixz="0"
-                    iyy="1E-6" iyz="0"
-                    izz="1E-6" />
-        </inertial>
-        <visual>
-            <origin  xyz="0 0 0"  rpy="0 0 0" />
-            <geometry>
-                <mesh filename="package://scara_v2_with_gripper/meshes/GripperBase.STL" />
-            </geometry>
-            <material name="sensoDarkGray">
-               <!-- <color rgba="0.792156862745098 0.819607843137255 0.933333333333333 1" />-->
-            </material>
-        </visual>
-        <collision>
-            <origin xyz="0 0 0" rpy="0 0 0" />
-            <geometry>
-                <mesh filename="package://scara_v2_with_gripper/meshes/GripperBase.STL" />
-            </geometry>
-        </collision>
-    </link>
-    <joint name="Joint_GripperBase" type="prismatic">
-        <parent link="ScaraLink2" />
-        <child link="GripperBase" />
-        <origin xyz="0 -0.0424 0.24305" rpy="3.1416 0 3.1416" />
-        <axis xyz="0 1 0" />
-        <limit effort="1000.0" lower="-0.03" upper="0.03" velocity="1"/>
-    </joint>
-    <link name="GripperLeft">
-        <inertial>
-            <origin  xyz="0 0 0"  rpy="3.14 0 0" />
-            <mass value="1" />
-            <inertia ixx="1E-6"  ixy="0" ixz="0"
-                    iyy="1E-6" iyz="0"
-                    izz="1E-6" />
-        </inertial>
-        <visual>
-            <origin xyz="0 0 0" rpy="3.14 0 0" />
-            <geometry>
-                <mesh filename="package://scara_v2_with_gripper/meshes/gripperLeft_full.STL" />
-            </geometry>
-            <material name="sensoDarkGray">
-            </material>
-        </visual>
-        <collision>
-            <origin xyz="0 0 0" rpy="0 0 0" />
-            <geometry>
-                <mesh  filename="package://scara_v2_with_gripper/meshes/gripperLeft_full.STL" />
-            </geometry>
-        </collision>
-    </link>
-    <joint name="Joint_Gripper" type="prismatic">
-        <parent link="GripperBase" />
-        <child link="GripperLeft" />
-        <origin xyz="-0.0162 0.0984 0" rpy="3.1416 0 0" />
-        <axis xyz="1 0 0" />
-        <limit effort="1000.0" lower="0" upper="0.003" velocity="1"/>
-    </joint>
-    <link name="GripperRight">
-        <inertial>
-            <origin   xyz="0 0 0" rpy="3.14 0 0" />
-            <mass value="1" />
-            <inertia  ixx="1E-6"  ixy="0" ixz="0"
-                    iyy="1E-6" iyz="0"
-                    izz="1E-6" />
-        </inertial>
-        <visual>
-            <origin  xyz="0 0 0"  rpy="3.14 0 0" />
-            <geometry>
-                <mesh filename="package://scara_v2_with_gripper/meshes/gripperRight_full.STL" />
-            </geometry>
-            <material name="sensoDarkGray">
-            </material>
-        </visual>
-        <collision>
-            <origin  xyz="0 0 0" rpy="0 0 0" />
-            <geometry>
-                <mesh  filename="package://scara_v2_with_gripper/meshes/gripperRight_full.STL" />
-            </geometry>
-        </collision>
-    </link>
-    <joint name="Joint_GripperRight" type="prismatic">
-        <parent link="GripperBase" />
-        <child link="GripperRight" />
-        <origin  xyz="0.0165 0.0984 0" rpy="3.1416 0 3.1416" />
-        <axis  xyz="1 0 0" />
-        <limit effort="1000.0" lower="-0.003" upper="0.003" velocity="1"/>
-        <mimic joint="Joint_Gripper" multiplier="1" offset="0" />
-    </joint>
-    <!--     Transmision definitions      -->
+    <!--
+     <link name="GripperBase">
+         <inertial>
+             <origin xyz="0 0 0" rpy="0 0 0" />
+             <mass  value="1" />
+             <inertia  ixx="1E-6" ixy="0" ixz="0"
+                     iyy="1E-6" iyz="0"
+                     izz="1E-6" />
+         </inertial>
+         <visual>
+             <origin  xyz="0 0 0"  rpy="0 0 0" />
+             <geometry>
+                 <mesh filename="package://scara_v2_with_gripper/meshes/GripperBase.STL" />
+             </geometry>
+             <material name="sensoDarkGray">
+             </material>
+         </visual>
+         <collision>
+             <origin xyz="0 0 0" rpy="0 0 0" />
+             <geometry>
+                 <mesh filename="package://scara_v2_with_gripper/meshes/GripperBase.STL" />
+             </geometry>
+         </collision>
+     </link>
+     <joint name="Joint_GripperBase" type="prismatic">
+         <parent link="ScaraLink2" />
+         <child link="GripperBase" />
+         <origin xyz="0 -0.0424 0.24305" rpy="3.1416 0 3.1416" />
+         <axis xyz="0 1 0" />
+         <limit effort="1000.0" lower="-0.03" upper="0.03" velocity="1"/>
+     </joint>
+     <link name="GripperLeft">
+         <inertial>
+             <origin  xyz="0 0 0"  rpy="3.14 0 0" />
+             <mass value="1" />
+             <inertia ixx="1E-6"  ixy="0" ixz="0"
+                     iyy="1E-6" iyz="0"
+                     izz="1E-6" />
+         </inertial>
+         <visual>
+             <origin xyz="0 0 0" rpy="3.14 0 0" />
+             <geometry>
+                 <mesh filename="package://scara_v2_with_gripper/meshes/gripperLeft_full.STL" />
+             </geometry>
+             <material name="sensoDarkGray">
+             </material>
+         </visual>
+         <collision>
+             <origin xyz="0 0 0" rpy="0 0 0" />
+             <geometry>
+                 <mesh  filename="package://scara_v2_with_gripper/meshes/gripperLeft_full.STL" />
+             </geometry>
+         </collision>
+     </link>
+     <joint name="Joint_Gripper" type="prismatic">
+         <parent link="GripperBase" />
+         <child link="GripperLeft" />
+         <origin xyz="-0.0162 0.0984 0" rpy="3.1416 0 0" />
+         <axis xyz="1 0 0" />
+         <limit effort="1000.0" lower="0" upper="0.003" velocity="1"/>
+     </joint>
+     <link name="GripperRight">
+         <inertial>
+             <origin   xyz="0 0 0" rpy="3.14 0 0" />
+             <mass value="1" />
+             <inertia  ixx="1E-6"  ixy="0" ixz="0"
+                     iyy="1E-6" iyz="0"
+                     izz="1E-6" />
+         </inertial>
+         <visual>
+             <origin  xyz="0 0 0"  rpy="3.14 0 0" />
+             <geometry>
+                 <mesh filename="package://scara_v2_with_gripper/meshes/gripperRight_full.STL" />
+             </geometry>
+             <material name="sensoDarkGray">
+             </material>
+         </visual>
+         <collision>
+             <origin  xyz="0 0 0" rpy="0 0 0" />
+             <geometry>
+                 <mesh  filename="package://scara_v2_with_gripper/meshes/gripperRight_full.STL" />
+             </geometry>
+         </collision>
+     </link>
+     <joint name="Joint_GripperRight" type="prismatic">
+         <parent link="GripperBase" />
+         <child link="GripperRight" />
+         <origin  xyz="0.0165 0.0984 0" rpy="3.1416 0 3.1416" />
+         <axis  xyz="1 0 0" />
+         <limit effort="1000.0" lower="-0.003" upper="0.003" velocity="1"/>
+         <mimic joint="Joint_Gripper" multiplier="1" offset="0" />
+     </joint>
+     -->
+     <!--     Transmision definitions      -->
     <transmission name="tran1">
         <type>transmission_interface/SimpleTransmission</type>
@@ -292,5 +294,5 @@
         <actuator name="motor1">
             <hardwareInterface>EffortJointInterface</hardwareInterface>
-            <mechanicalReduction>1</mechanicalReduction>
+            <mechanicalReduction>1000</mechanicalReduction>
         </actuator>
     </transmission>
@@ -302,7 +304,8 @@
         <actuator name="motor2">
             <hardwareInterface>EffortJointInterface</hardwareInterface>
-            <mechanicalReduction>1</mechanicalReduction>
+            <mechanicalReduction>1000</mechanicalReduction>
         </actuator>
     </transmission>
+    <!--
     <transmission name="tran3">
         <type>transmission_interface/SimpleTransmission</type>
@@ -312,5 +315,5 @@
         <actuator name="motor3">
             <hardwareInterface>EffortJointInterface</hardwareInterface>
-            <mechanicalReduction>1</mechanicalReduction>
+            <mechanicalReduction>1000</mechanicalReduction>
         </actuator>
     </transmission>
@@ -322,7 +325,8 @@
         <actuator name="motor4">
             <hardwareInterface>EffortJointInterface</hardwareInterface>
-            <mechanicalReduction>1</mechanicalReduction>
+            <mechanicalReduction>1000</mechanicalReduction>
         </actuator>
     </transmission>
+    -->
     <!-- ***************************** -->
 </robot>
