Commit message: scara and rotary table RViz and MoveIt! config

File: gazebo_scara_v2_with_gripper/scara_v2_description/urdf/scara_v2_urdf.xacro (robot description, xacro)
@@ -193,34 +193,34 @@
     <!--**********************************-->
     <!--     GRIPPER JOINTS DEFINITION    -->
-     <!--<link name="GripperBase">-->
-         <!--<inertial>-->
-             <!--<origin xyz="0 0 0" rpy="0 0 0" />-->
-             <!--<mass  value="1" />-->
-             <!--<inertia  ixx="1E-6" ixy="0" ixz="0"-->
-                     <!--iyy="1E-6" iyz="0"-->
-                     <!--izz="1E-6" />-->
-         <!--</inertial>-->
-         <!--<visual>-->
-             <!--<origin  xyz="0 0 0"  rpy="0 0 0" />-->
-             <!--<geometry>-->
-                 <!--<mesh filename="package://scara_v2_with_gripper/meshes/GripperBase.STL" />-->
-             <!--</geometry>-->
-             <!--<material name="sensoDarkGray">-->
-             <!--</material>-->
-         <!--</visual>-->
-         <!--<collision>-->
-             <!--<origin xyz="0 0 0" rpy="0 0 0" />-->
-             <!--<geometry>-->
-                 <!--<mesh filename="package://scara_v2_with_gripper/meshes/GripperBase.STL" />-->
-             <!--</geometry>-->
-         <!--</collision>-->
-     <!--</link>-->
-     <!--<joint name="Joint_GripperBase" type="prismatic">-->
-         <!--<parent link="ScaraLink2" />-->
-         <!--<child link="GripperBase" />-->
-         <!--<origin xyz="0 -0.0424 0.24305" rpy="3.1416 0 3.1416" />-->
-         <!--<axis xyz="0 1 0" />-->
-         <!--<limit effort="1000.0" lower="-0.04" upper="0.05" velocity="1"/>-->
-     <!--</joint>-->
+     <link name="GripperBase">
+         <inertial>
+             <origin xyz="0 0 0" rpy="0 0 0" />
+             <mass  value="1" />
+             <inertia  ixx="1E-6" ixy="0" ixz="0"
+                     iyy="1E-6" iyz="0"
+                     izz="1E-6" />
+         </inertial>
+         <visual>
+             <origin  xyz="0 0 0"  rpy="0 0 0" />
+             <geometry>
+                 <mesh filename="package://scara_v2_with_gripper/meshes/GripperBase.STL" />
+             </geometry>
+             <material name="sensoDarkGray">
+             </material>
+         </visual>
+         <collision>
+             <origin xyz="0 0 0" rpy="0 0 0" />
+             <geometry>
+                 <mesh filename="package://scara_v2_with_gripper/meshes/GripperBase.STL" />
+             </geometry>
+         </collision>
+     </link>
+     <joint name="Joint_GripperBase" type="prismatic">
+         <parent link="ScaraLink2" />
+         <child link="GripperBase" />
+         <origin xyz="0 -0.0424 0.24305" rpy="3.1416 0 3.1416" />
+         <axis xyz="0 1 0" />
+         <limit effort="1000.0" lower="-0.04" upper="0.05" velocity="1"/>
+     </joint>
      <!--<link name="GripperLeft">-->
          <!--<inertial>-->
