Commit message: moveit_API_2 with new moveit_config

File: scara_v2_with_gripper/urdf/scara_v2_with_gripper.urdf (robot description, URDF)
Before this commit: robot scara_v2_with_gripper, 9 links, 8 joints
Links:
- added link tool0
- added link world
- link ScaraLink1: mass 1 -> 3.8063
- link ScaraLink2: mass 1 -> 1.5020
Joints:
- added joint Base_to_tool0: type fixed, parent GripperBase, child tool0, origin xyz=0 0.0984 0 rpy=0 0 0 
- added joint world_to_BaseBox: type fixed, parent world, child BaseBox, origin xyz=0 0 0.965 rpy=0 0 0, axis 1 0 0
- joint Joint1: limit lower=-1.57079 upper=1.57079 effort=0 velocity=0 -> lower=-1.4835298642 upper=1.4835298642 effort=0 velocity=0
- joint Joint2: limit lower=-2.65 upper=2.65 effort=0 velocity=0 -> lower=-2.9670597284 upper=2.9670597284 effort=0 velocity=0
- joint Joint_GripperRight: limit lower=-0.003 upper=0.003 effort=1000.0 velocity=1 -> lower=0 upper=0.003 effort=1000.0 velocity=1; mimic joint=Joint_Gripper multiplier=1 offset=0 -> (none)

File: scara_v2_with_gripper/urdf/scara_v2_with_gripper_urdf.xacro (robot description, xacro)
@@ -1,4 +1,4 @@
 <?xml version="1.0"?>
-<robot  name="scara_v2_with_gripper">
+<robot  name="scara_v2" xmlns:xacro="http://www.ros.org/wiki/xacro">
     <!--  Material Color definitions -->
     <material name="white">
@@ -26,4 +26,8 @@
         <color rgba="0.156863 0.156863 0.156863 1 "/>
     </material>
+    <!--****************************-->
+    <!--**********MACROS************-->
+    <xacro:property name="DEG2RAD" value="0.01745329252" />
+    <xacro:property name="RED2DEG" value="57.295779513" />
     <!--****************************-->
     <!-- Link and Joint definitions  -->
@@ -181,5 +185,6 @@
         <origin xyz="0 0.051 0" rpy="0 0 0" />
         <axis xyz="0 1 0" />
-        <limit effort="0" lower="-1.57079" upper="1.57079" velocity="0"/>
+        <!--<limit effort="0" lower="-1.57079" upper="1.57079" velocity="0"/>-->
+        <limit effort="0" lower="${-85*DEG2RAD}" upper="${85*DEG2RAD}" velocity="0"/>
     </joint>
     <link name="ScaraLink2">
@@ -212,5 +217,6 @@
         <origin xyz="0.24972 -0.081 0" rpy="3.14 -1.5708 0" />
         <axis xyz="0 1 0" />
-        <limit effort="0" lower="-2.65" upper="2.65" velocity="0"/>
+        <!--<limit effort="0" lower="-2.65" upper="2.65" velocity="0"/>-->
+        <limit effort="0" lower="${-170*DEG2RAD}" upper="${170*DEG2RAD}" velocity="0"/>
     </joint>
     <!--**********************************-->
@@ -247,4 +253,10 @@
         <limit effort="1000.0" lower="-0.03" upper="0.03" velocity="1"/>
     </joint>
+    <joint name="Base_to_tool0" type="fixed">
+        <parent link="GripperBase" />
+        <child link="tool0" />
+        <origin xyz="0 0.0984 0" rpy="0 0 0 " />
+    </joint>
+    <link name="tool0"/>
     <link name="GripperLeft">
         <inertial>
@@ -307,6 +319,6 @@
         <origin  xyz="0.0165 0.0984 0" rpy="3.1416 0 3.1416" />
         <axis  xyz="1 0 0" />
-        <limit effort="1000.0" lower="-0.003" upper="0.003" velocity="1"/>
-        <mimic joint="Joint_Gripper" multiplier="1" offset="0" />
+        <limit effort="1000.0" lower="0" upper="0.003" velocity="1"/>
+        <!--<mimic joint="Joint_Gripper" multiplier="1" offset="0" />-->
     </joint>
 </robot>
