Commit message: snaha o novy ikfast s upravenym urdf

File: scara_v2_with_gripper/urdf/scara_v2_with_gripper_urdf.urdf (robot description, URDF)
Before this commit: robot scara_v2, 12 links, 11 joints
Joints:
- joint Joint1: axis 0 1 0 -> 0 0 1; origin xyz=0 0.051 0 rpy=0 0 0 -> xyz=0 0.051 0 rpy=1.57 0 0
- joint Joint2: axis 0 1 0 -> 0 0 1; origin xyz=0.24972 -0.081 0 rpy=3.14 -1.5708 0 -> xyz=0.24972  0 0.081 rpy=0 0 0
- joint fake_joint: origin xyz=0 -0.0424 0.24305 rpy=1.57 0 3.1416 -> xyz=0 -0.24305 -0.0424  rpy=0 0 3.1416

File: scara_v2_with_gripper/urdf/scara_v2_with_gripper_urdf.xacro (robot description, xacro)
@@ -155,5 +155,5 @@
     <link name="ScaraLink1">
         <inertial>
-            <origin xyz="0 0 0" rpy="0 0 0" />
+            <origin xyz="0 0 0" rpy="-1.57 0 0" />
             <mass value="3.8063" />
             <inertia ixx="7.8753E-3" ixy="4.6431E-3" ixz="-1.4702E-5"
@@ -162,5 +162,5 @@
         </inertial>
         <visual>
-            <origin xyz="0 0 0" rpy="0 0 0" />
+            <origin xyz="0 0 0" rpy="-1.57 0 0" />
             <geometry>
                 <mesh filename="package://scara_v2_with_gripper/meshes/ScaraLink1.STL" />   <!--ScaraLink1.STL-->
@@ -170,5 +170,5 @@
         </visual>
         <collision>
-            <origin xyz="0 0 0" rpy="0 0 0" />
+            <origin xyz="0 0 0" rpy="-1.57 0 0" />
             <geometry>
                 <mesh filename="package://scara_v2_with_gripper/meshes/ScaraLink1.STL" />
@@ -179,6 +179,6 @@
         <parent link="ScaraBase" />
         <child link="ScaraLink1" />
-        <origin xyz="0 0.051 0" rpy="0 0 0" />
-        <axis xyz="0 1 0" />
+        <origin xyz="0 0.051 0" rpy="1.57 0 0" />
+        <axis xyz="0 0 1" />
         <!--<limit effort="0" lower="-1.57079" upper="1.57079" velocity="0"/>-->
         <limit effort="0" lower="${-85*DEG2RAD}" upper="${85*DEG2RAD}" velocity="0"/>
@@ -186,5 +186,5 @@
     <link name="ScaraLink2">
         <inertial>
-            <origin xyz="0 0 0" rpy="0 0 0" />
+            <origin xyz="0 0 0" rpy="1.57 1.57 0" />
             <mass value="1.5020" />
             <inertia  ixx="5.0471E-2" ixy="3.0689E-4" ixz="-8.5622E-4"
@@ -193,5 +193,5 @@
         </inertial>
         <visual>
-            <origin  xyz="0 0 0" rpy="0 0 0" />
+            <origin  xyz="0 0 0" rpy="1.57 0 0" />
             <geometry>
                 <mesh  filename="package://scara_v2_with_gripper/meshes/ScaraLink2.STL" />
@@ -201,5 +201,5 @@
         </visual>
         <collision>
-            <origin xyz="0 0 0" rpy="0 0 0" />
+            <origin xyz="0 0 0" rpy="0 1.57 0" />
             <geometry>
                 <mesh filename="package://scara_v2_with_gripper/meshes/ScaraLink2.STL" />
@@ -210,6 +210,6 @@
         <parent link="ScaraLink1" />
         <child link="ScaraLink2" />
-        <origin xyz="0.24972 -0.081 0" rpy="3.14 -1.5708 0" />
-        <axis xyz="0 1 0" />
+        <origin xyz="0.24972  0 0.081" rpy="0 0 0" />
+        <axis xyz="0 0 1" />
         <!--<limit effort="0" lower="-2.65" upper="2.65" velocity="0"/>-->
         <limit effort="0" lower="${-170*DEG2RAD}" upper="${170*DEG2RAD}" velocity="0"/>
@@ -222,5 +222,6 @@
         <parent link="ScaraLink2" />
         <child link="fake_link" />
-        <origin xyz="0 -0.0424 0.24305" rpy="1.57 0 3.1416" />
+        <!--<origin xyz="0 -0.24305 0.0424 " rpy="0 0 3.1416" />-->
+        <origin xyz="0 -0.24305 -0.0424 " rpy="0 0 3.1416" />
         <axis xyz="0 0 1" />
         <limit effort="1000.0" lower="0.0" upper="0.001" velocity="0"/>
