Commit message: IK fast service start

File: scara_v2_with_gripper/urdf/scara_v2_with_gripper_urdf.xacro (robot description, xacro)
@@ -54,11 +54,11 @@
             </geometry>
             <material name="sensoGray">
-              <!--  <color rgba="0.792156862745098 0.819607843137255 0.933333333333333 1" />-->
-            </material>
-        </visual>
-        <collision>
-            <origin xyz="0 0 0" rpy="0 0 0" />
-            <geometry>
-                <mesh filename="package://scara_v2_with_gripper/meshes/baseBox.STL" />
+            </material>
+        </visual>
+        <collision>
+            <origin xyz="0 0 0" rpy="0 0 0" />
+            <geometry>
+                <!--?????????-->
+                <mesh filename="package://scara_v2_with_gripper/meshes/baseBox_modif.stl" />
             </geometry>
         </collision>
@@ -78,11 +78,10 @@
             </geometry>
             <material name="red">
-                <!--<color rgba="0.792156862745098 0.819607843137255 0.933333333333333 1" />-->
-            </material>
-        </visual>
-        <collision>
-            <origin xyz="0 0 0" rpy="0 0 0" />
-            <geometry>
-                <mesh filename="package://scara_v2_with_gripper/meshes/CentralStop1.STL" />
+            </material>
+        </visual>
+        <collision>
+            <origin xyz="0 0 0" rpy="0 0 0" />
+            <geometry>
+                <mesh filename="package://scara_v2_with_gripper/meshes/CentralStop1_modif.stl" />
             </geometry>
         </collision>
@@ -108,11 +107,10 @@
             </geometry>
             <material name="red">
-                <!--<color rgba="0.792156862745098 0.819607843137255 0.933333333333333 1" />-->
-            </material>
-        </visual>
-        <collision>
-            <origin xyz="0 0 0" rpy="0 0 0" />
-            <geometry>
-                <mesh filename="package://scara_v2_with_gripper/meshes/CentralStop2.STL" />
+            </material>
+        </visual>
+        <collision>
+            <origin xyz="0 0 0" rpy="0 0 0" />
+            <geometry>
+                <mesh filename="package://scara_v2_with_gripper/meshes/CentralStop2_modif.stl" />
             </geometry>
         </collision>
@@ -140,5 +138,4 @@
             </geometry>
             <material  name="sensoSilver">
-                <!--<color rgba="0.792156862745098 0.819607843137255 0.933333333333333 1" />-->
             </material>
         </visual>
@@ -167,8 +164,7 @@
             <origin xyz="0 0 0" rpy="0 0 0" />
             <geometry>
-                <mesh filename="package://scara_v2_with_gripper/meshes/ScaraLink1.STL" />
+                <mesh filename="package://scara_v2_with_gripper/meshes/ScaraLink1.STL" />   <!--ScaraLink1.STL-->
             </geometry>
             <material name="sensoSilver">
-                <!--<color  rgba="0.79216 0.81961 0.93333 1" />-->
             </material>
         </visual>
@@ -202,5 +198,4 @@
             </geometry>
             <material  name="sensoSilver">
-                <!--<color rgba="0.79216 0.81961 0.93333 1" />-->
             </material>
         </visual>
@@ -236,5 +231,4 @@
             </geometry>
             <material name="sensoDarkGray">
-               <!-- <color rgba="0.792156862745098 0.819607843137255 0.933333333333333 1" />-->
             </material>
         </visual>
@@ -251,5 +245,5 @@
         <origin xyz="0 -0.0424 0.24305" rpy="3.1416 0 3.1416" />
         <axis xyz="0 1 0" />
-        <limit effort="1000.0" lower="-0.03" upper="0.03" velocity="1"/>
+        <limit effort="1000.0" lower="-0.04" upper="0.05" velocity="1"/>
     </joint>
     <joint name="Base_to_tool0" type="fixed">
@@ -273,9 +267,8 @@
             </geometry>
             <material name="sensoDarkGray">
-               <!-- <color  rgba="0.79216 0.81961 0.93333 1" />-->
-            </material>
-        </visual>
-        <collision>
-            <origin xyz="0 0 0" rpy="0 0 0" />
+            </material>
+        </visual>
+        <collision>
+            <origin xyz="0 0 0" rpy="3.14 0 0" />
             <geometry>
                 <mesh  filename="package://scara_v2_with_gripper/meshes/gripperLeft_full.STL" />
@@ -304,9 +297,8 @@
             </geometry>
             <material name="sensoDarkGray">
-                <!--<color  rgba="0.79216 0.81961 0.93333 1" />-->
-            </material>
-        </visual>
-        <collision>
-            <origin  xyz="0 0 0" rpy="0 0 0" />
+            </material>
+        </visual>
+        <collision>
+            <origin  xyz="0 0 0" rpy="3.14 0 0" />
             <geometry>
                 <mesh  filename="package://scara_v2_with_gripper/meshes/gripperRight_full.STL" />
@@ -320,5 +312,5 @@
         <axis  xyz="1 0 0" />
         <limit effort="1000.0" lower="0" upper="0.003" velocity="1"/>
-        <!--<mimic joint="Joint_Gripper" multiplier="1" offset="0" />-->
+        <mimic joint="Joint_Gripper" multiplier="1" offset="0" />
     </joint>
 </robot>

Commit message: position and joint control v.1
Signed-off-by: dluhosko@gmail.com <dluhosko>

File: scara_v2_with_gripper/urdf/scara_v2_with_gripper_urdf.xacro (robot description, xacro)
@@ -201,5 +201,5 @@
         </visual>
         <collision>
-            <origin xyz="0 0 0" rpy="0 1.57 0" />
+            <origin xyz="0 0 0" rpy="1.57 0 0" />
             <geometry>
                 <mesh filename="package://scara_v2_with_gripper/meshes/ScaraLink2.STL" />
