Commit message: snaha o novy ikfast

File: scara_v2_with_gripper/urdf/scara_and_rt_urdf.xacro (robot description, xacro)
@@ -790,7 +790,17 @@
     <!--**********************************-->
     <!--     GRIPPER JOINTS DEFINITION    -->
+    <!--     GRIPPER JOINTS DEFINITION    -->
+    <!--Revolute joint for IKfast-->
+    <link name="fake_link"/>
+    <joint name="fake_joint" type="revolute">
+        <parent link="ScaraLink2" />
+        <child link="fake_link" />
+        <origin xyz="0 -0.0424 0.24305" rpy="1.57 0 3.1416" />
+        <axis xyz="0 0 1" />
+        <limit effort="1000.0" lower="0.0" upper="0.001" velocity="0"/>
+    </joint>
     <link name="GripperBase">
         <inertial>
-            <origin xyz="0 0 0" rpy="0 0 0" />
+            <origin xyz="0 0 0" rpy="1.57 0 0" />
             <mass  value="1" />
             <inertia  ixx="1E-6" ixy="0" ixz="0"
@@ -799,5 +809,5 @@
         </inertial>
         <visual>
-            <origin  xyz="0 0 0"  rpy="0 0 0" />
+            <origin  xyz="0 0 0"  rpy="1.57 0 0" />
             <geometry>
                 <mesh filename="package://scara_v2_with_gripper/meshes/GripperBase.STL" />
@@ -807,5 +817,5 @@
         </visual>
         <collision>
-            <origin xyz="0 0 0" rpy="0 0 0" />
+            <origin xyz="0 0 0" rpy="1.57 0 0" />
             <geometry>
                 <mesh filename="package://scara_v2_with_gripper/meshes/GripperBase.STL" />
@@ -814,16 +824,18 @@
     </link>
     <joint name="Joint_GripperBase" type="prismatic">
-        <parent link="ScaraLink2" />
+        <parent link="fake_link" />
         <child link="GripperBase" />
-        <origin xyz="0 -0.0424 0.24305" rpy="3.1416 0 3.1416" />
-        <axis xyz="0 1 0" />
+        <origin xyz="0 0 0" rpy="0 0 0" />
+        <!--<origin xyz="0 -0.0424 0.24305" rpy="3.1416 0 3.1416" />-->
+        <axis xyz="0 0 1" />
         <limit effort="1000.0" lower="-0.04" upper="0.05" velocity="1"/>
     </joint>
+    <link name="tool0"/>
     <joint name="Base_to_tool0" type="fixed">
         <parent link="GripperBase" />
         <child link="tool0" />
-        <origin xyz="0 0.0984 0" rpy="0 0 0 " />
-    </joint>
-    <link name="tool0"/>
+        <origin xyz="0 0 0.0984" rpy="0 0 0 " />
+        <axis xyz="0 0 0" />
+    </joint>
     <link name="GripperLeft">
         <inertial>
@@ -852,5 +864,5 @@
         <parent link="GripperBase" />
         <child link="GripperLeft" />
-        <origin xyz="-0.0162 0.0984 0" rpy="3.1416 0 0" />
+        <origin xyz="-0.0162 0 0.0984" rpy="-1.57 0 0" />
         <axis xyz="1 0 0" />
         <limit effort="1000.0" lower="0" upper="0.003" velocity="1"/>
@@ -882,5 +894,5 @@
         <parent link="GripperBase" />
         <child link="GripperRight" />
-        <origin  xyz="0.0165 0.0984 0" rpy="3.1416 0 3.1416" />
+        <origin  xyz="0.0165 0 0.0984" rpy="1.57 0 3.1416" />
         <axis  xyz="1 0 0" />
         <limit effort="1000.0" lower="0" upper="0.003" velocity="1"/>

File: scara_v2_with_gripper/urdf/scara_v2_with_gripper_urdf.xacro (robot description, xacro)
@@ -217,7 +217,16 @@
     <!--**********************************-->
     <!--     GRIPPER JOINTS DEFINITION    -->
+    <!--Revolute joint for IKfast-->
+    <link name="fake_link"/>
+    <joint name="fake_joint" type="revolute">
+        <parent link="ScaraLink2" />
+        <child link="fake_link" />
+        <origin xyz="0 -0.0424 0.24305" rpy="1.57 0 3.1416" />
+        <axis xyz="0 0 1" />
+        <limit effort="1000.0" lower="0.0" upper="0.001" velocity="0"/>
+    </joint>
     <link name="GripperBase">
         <inertial>
-            <origin xyz="0 0 0" rpy="0 0 0" />
+            <origin xyz="0 0 0" rpy="1.57 0 0" />
             <mass  value="1" />
             <inertia  ixx="1E-6" ixy="0" ixz="0"
@@ -226,5 +235,5 @@
         </inertial>
         <visual>
-            <origin  xyz="0 0 0"  rpy="0 0 0" />
+            <origin  xyz="0 0 0"  rpy="1.57 0 0" />
             <geometry>
                 <mesh filename="package://scara_v2_with_gripper/meshes/GripperBase.STL" />
@@ -234,5 +243,5 @@
         </visual>
         <collision>
-            <origin xyz="0 0 0" rpy="0 0 0" />
+            <origin xyz="0 0 0" rpy="1.57 0 0" />
             <geometry>
                 <mesh filename="package://scara_v2_with_gripper/meshes/GripperBase.STL" />
@@ -241,16 +250,18 @@
     </link>
     <joint name="Joint_GripperBase" type="prismatic">
-        <parent link="ScaraLink2" />
+        <parent link="fake_link" />
         <child link="GripperBase" />
-        <origin xyz="0 -0.0424 0.24305" rpy="3.1416 0 3.1416" />
-        <axis xyz="0 1 0" />
+        <origin xyz="0 0 0" rpy="0 0 0" />
+        <!--<origin xyz="0 -0.0424 0.24305" rpy="3.1416 0 3.1416" />-->
+        <axis xyz="0 0 1" />
         <limit effort="1000.0" lower="-0.04" upper="0.05" velocity="1"/>
     </joint>
+    <link name="tool0"/>
     <joint name="Base_to_tool0" type="fixed">
         <parent link="GripperBase" />
         <child link="tool0" />
-        <origin xyz="0 0.0984 0" rpy="0 0 0 " />
-    </joint>
-    <link name="tool0"/>
+        <origin xyz="0 0 0.0984" rpy="0 0 0 " />
+        <axis xyz="0 0 0" />
+    </joint>
     <link name="GripperLeft">
         <inertial>
@@ -279,5 +290,5 @@
         <parent link="GripperBase" />
         <child link="GripperLeft" />
-        <origin xyz="-0.0162 0.0984 0" rpy="3.1416 0 0" />
+        <origin xyz="-0.0162 0 0.0984" rpy="-1.57 0 0" />
         <axis xyz="1 0 0" />
         <limit effort="1000.0" lower="0" upper="0.003" velocity="1"/>
@@ -309,5 +320,5 @@
         <parent link="GripperBase" />
         <child link="GripperRight" />
-        <origin  xyz="0.0165 0.0984 0" rpy="3.1416 0 3.1416" />
+        <origin  xyz="0.0165 0 0.0984" rpy="1.57 0 3.1416" />
         <axis  xyz="1 0 0" />
         <limit effort="1000.0" lower="0" upper="0.003" velocity="1"/>

Commit message: position and joint control v.1 (upraveny moveit)
Signed-off-by: dluhosko@gmail.com <dluhosko>

File: scara_v2_with_gripper/urdf/scara_and_rt_urdf.xacro (robot description, xacro)
@@ -792,12 +792,12 @@
     <!--     GRIPPER JOINTS DEFINITION    -->
     <!--Revolute joint for IKfast-->
-    <link name="fake_link"/>
-    <joint name="fake_joint" type="revolute">
-        <parent link="ScaraLink2" />
-        <child link="fake_link" />
-        <origin xyz="0 -0.0424 0.24305" rpy="1.57 0 3.1416" />
-        <axis xyz="0 0 1" />
-        <limit effort="1000.0" lower="0.0" upper="0.001" velocity="0"/>
-    </joint>
+    <!--<link name="fake_link"/>-->
+    <!--<joint name="fake_joint" type="revolute">-->
+        <!--<parent link="ScaraLink2" />-->
+        <!--<child link="fake_link" />-->
+        <!--<origin xyz="0 -0.0424 0.24305" rpy="1.57 0 3.1416" />-->
+        <!--<axis xyz="0 0 1" />-->
+        <!--<limit effort="1000.0" lower="0.0" upper="0.001" velocity="0"/>-->
+    <!--</joint>-->
     <link name="GripperBase">
         <inertial>
@@ -824,8 +824,8 @@
     </link>
     <joint name="Joint_GripperBase" type="prismatic">
-        <parent link="fake_link" />
+        <parent link="ScaraLink2" />
         <child link="GripperBase" />
-        <origin xyz="0 0 0" rpy="0 0 0" />
-        <!--<origin xyz="0 -0.0424 0.24305" rpy="3.1416 0 3.1416" />-->
+        <!--<origin xyz="0 0 0" rpy="0 0 0" />-->
+        <origin xyz="0 -0.0424 0.24305" rpy="1.57 0 3.1416" />
         <axis xyz="0 0 1" />
         <limit effort="1000.0" lower="-0.04" upper="0.05" velocity="1"/>

Commit message: linearna interpolacia proste nejde...
Signed-off-by: senso-viktor <viktordluhos@gmail.com>

File: scara_v2_with_gripper/urdf/scara_and_rt_urdf.xacro (robot description, xacro)
@@ -30,4 +30,5 @@
     <xacro:property name="DEG2RAD" value="0.01745329252" />
     <xacro:property name="RED2DEG" value="57.295779513" />
+    <xacro:property name="M_PI" value="3.141592" />
     <!--****************************-->
     <!-- Link and Joint definitions  -->
@@ -508,5 +509,5 @@
         <origin xyz="0 0 0.01" rpy="0 0 0"/>
         <axis xyz="0 0 1" />
-        <limit effort="1000" lower="0" upper="6.29" velocity="0"/>
+        <limit effort="1000" lower="0" upper="${2*M_PI}" velocity="0"/>
     </joint>
     <link name="hole1">
@@ -853,9 +854,11 @@
     </joint>
     <link name="tool0"/>
-    <joint name="Base_to_tool0" type="fixed">
+    <joint name="Base_to_tool0" type="revolute">
         <parent link="GripperBase" />
         <child link="tool0" />
         <origin xyz="0 0 0.0984" rpy="0 0 0 " />
-        <axis xyz="0 0 0" />
+        <axis xyz="0 0 1" />
+        <!--<limit effort="0" lower="-2.65" upper="2.65" velocity="0"/>-->
+        <limit effort="0" lower="${-M_PI}" upper="${M_PI}" velocity="0"/>
     </joint>
     <link name="GripperLeft">

Commit message: my pc + senso pc
Signed-off-by: senso-viktor <viktordluhos@gmail.com>

File: scara_v2_with_gripper/urdf/scara_and_rt_urdf.xacro (robot description, xacro)
@@ -30,5 +30,4 @@
     <xacro:property name="DEG2RAD" value="0.01745329252" />
     <xacro:property name="RED2DEG" value="57.295779513" />
-    <xacro:property name="M_PI" value="3.141592" />
     <!--****************************-->
     <!-- Link and Joint definitions  -->
@@ -154,33 +153,33 @@
     </joint>
     <!--_______Colision object_______-->
-    <!--<link name="colisionBox">-->
-        <!--<inertial>-->
-            <!--<origin xyz="0 0 0" rpy="0 0 0" />-->
-            <!--<mass value="1" />-->
-            <!--<inertia ixx="1" ixy="0" ixz="0"-->
-                     <!--iyy="1" iyz="0"-->
-                     <!--izz="1" />-->
-        <!--</inertial>-->
-        <!--<visual>-->
-            <!--<origin xyz="0 0 0" rpy="0 0 0" />-->
-            <!--<geometry>-->
-                <!--<box size="0.05 0.05 0.2"/>-->
-            <!--</geometry>-->
-            <!--<material name="sensoSilver">-->
-            <!--</material>-->
-        <!--</visual>-->
-        <!--<collision>-->
-            <!--<origin xyz="0 0 0" rpy="0 0 0" />-->
-            <!--<geometry>-->
-                <!--<box size="0.1 0.1 0.2"/>-->
-            <!--</geometry>-->
-        <!--</collision>-->
-    <!--</link>-->
-    <!--<joint name="Joint_colisionBox" type="fixed">-->
-        <!--<parent link="BaseBox" />-->
-        <!--<child link="colisionBox" />-->
-        <!--<origin xyz="0.55 0.40 0.1" rpy="0 0 0" />-->
-        <!--<axis xyz="1 0 0" />-->
-    <!--</joint>-->
+    <link name="colisionBox">
+        <inertial>
+            <origin xyz="0 0 0" rpy="0 0 0" />
+            <mass value="1" />
+            <inertia ixx="1" ixy="0" ixz="0"
+                     iyy="1" iyz="0"
+                     izz="1" />
+        </inertial>
+        <visual>
+            <origin xyz="0 0 0" rpy="0 0 0" />
+            <geometry>
+                <box size="0.05 0.05 0.2"/>
+            </geometry>
+            <material name="red">
+            </material>
+        </visual>
+        <collision>
+            <origin xyz="0 0 0" rpy="0 0 0" />
+            <geometry>
+                <box size="0.1 0.1 0.2"/>
+            </geometry>
+        </collision>
+    </link>
+    <joint name="Joint_colisionBox" type="fixed">
+        <parent link="BaseBox" />
+        <child link="colisionBox" />
+        <origin xyz="0.55 0.40 0.1" rpy="0 0 0" />
+        <axis xyz="1 0 0" />
+    </joint>
     <!--**************************-->
     <link name="placeHole1">
@@ -509,5 +508,5 @@
         <origin xyz="0 0 0.01" rpy="0 0 0"/>
         <axis xyz="0 0 1" />
-        <limit effort="1000" lower="0" upper="${2*M_PI}" velocity="0"/>
+        <limit effort="1000" lower="0" upper="6.29" velocity="0"/>
     </joint>
     <link name="hole1">
@@ -854,11 +853,9 @@
     </joint>
     <link name="tool0"/>
-    <joint name="Base_to_tool0" type="revolute">
+    <joint name="Base_to_tool0" type="fixed">
         <parent link="GripperBase" />
         <child link="tool0" />
         <origin xyz="0 0 0.0984" rpy="0 0 0 " />
-        <axis xyz="0 0 1" />
-        <!--<limit effort="0" lower="-2.65" upper="2.65" velocity="0"/>-->
-        <limit effort="0" lower="${-M_PI}" upper="${M_PI}" velocity="0"/>
+        <axis xyz="0 0 0" />
     </joint>
     <link name="GripperLeft">
