Commit message: SENSO PC + MY PC sync  + get information tab completed!
Signed-off-by: senso-viktor <viktordluhos@gmail.com>

File: scara_v2_with_gripper/urdf/scara_and_rt_urdf.xacro (robot description, xacro)
@@ -172,5 +172,5 @@
             <origin xyz="0 0 0" rpy="0 0 0" />
             <geometry>
-                <box size="0.1 0.1 0.2"/>
+                <box size="0.07 0.07 0.2"/>
             </geometry>
         </collision>
@@ -425,305 +425,305 @@
     <!-- ******************************-->
     <!--______________PICK BOX__________________-->
-    <link name="base">
-        <inertial>
-            <origin xyz="0 0 0" rpy="0 0 0" />
-            <mass value="1" />
-            <inertia ixx="1" ixy="0" ixz="0"
-                     iyy="1" iyz="0"
-                     izz="1" />
-        </inertial>
-        <visual>
-            <origin xyz="0 0 0" rpy="0 0 0"/>
-            <geometry>
-                <box size="0.15 0.1 0.01"/>
-            </geometry>
-            <material name="sensoBlack" />
-        </visual>
-        <collision>
-            <origin xyz="0 0 0" rpy="0 0 0" />
-            <geometry>
-                <box size="0.15 0.1 0.02"/>
-            </geometry>
-        </collision>
-    </link>
-    <joint name="world_to_base" type="fixed">
-        <parent link="BaseBox"/>
-        <child link="base"/>
-        <origin xyz="0.40 0.15 0.005" rpy="0 0 ${90*DEG2RAD}" />
-        <axis xyz="1 0 0" />
-    </joint>
-    <link name="base_link1">
-        <inertial>
-            <origin xyz="0 0 0" rpy="0 0 0" />
-            <mass value="1" />
-            <inertia ixx="1" ixy="0" ixz="0"
-                     iyy="1" iyz="0"
-                     izz="1" />
-        </inertial>
-        <visual>
-            <origin xyz="0 0 0" rpy="0 0 0"/>
-            <geometry>
-                <cylinder length="0.01" radius="0.02"/>
-            </geometry>
-            <material name="sensoSilver" />
-        </visual>
-        <collision>
-            <origin xyz="0 0 0" rpy="0 0 0" />
-            <geometry>
-                <cylinder length="0.01" radius="0.02"/>
-            </geometry>
-        </collision>
-    </link>
-    <joint name="base_to_base_link1" type="fixed">
-        <parent link="base"/>
-        <child link="base_link1"/>
-        <origin xyz="0.05 0 0.01" rpy="0 0 0"/>
-        <axis xyz="0 0 1" />
-    </joint>
-    <link name="link1">
-        <inertial>
-            <origin xyz="0 0 0" rpy="0 0 0" />
-            <mass value="1" />
-            <inertia ixx="1" ixy="0" ixz="0"
-                     iyy="1" iyz="0"
-                     izz="1" />
-        </inertial>
-        <visual>
-            <origin xyz="0 0 0" rpy="0 0 0"/>
-            <geometry>
-                <cylinder length="0.01" radius="0.06"/>
-            </geometry>
-            <material name="sensoSilver" />
-        </visual>
-        <collision>
-            <origin xyz="0 0 0" rpy="0 0 0" />
-            <geometry>
-                <cylinder length="0.02" radius="0.06"/>
-            </geometry>
-        </collision>
-    </link>
-    <joint name="base_link1_to_link1" type="revolute"> <!-- rotary table joint-->
-        <parent link="base_link1"/>
-        <child link="link1"/>
-        <origin xyz="0 0 0.01" rpy="0 0 0"/>
-        <axis xyz="0 0 1" />
-        <limit effort="1000" lower="0" upper="6.29" velocity="0"/>
-    </joint>
-    <link name="hole1">
-        <inertial>
-            <origin xyz="0 0 0" rpy="0 0 0" />
-            <mass value="0.1" />
-            <inertia ixx="1E-9" ixy="0" ixz="0"
-                     iyy="1E-9" iyz="0"
-                     izz="1E-9" />
-        </inertial>
-        <visual>
-            <origin xyz="0 0 0" rpy="0 0 0"/>
-            <geometry>
-                <cylinder length="0.005" radius="0.01"/>
-            </geometry>
-            <material name="blue" />
-        </visual>
-        <collision>
-            <origin xyz="0 0 0" rpy="0 0 0" />
-            <geometry>
-                <cylinder length="0.005" radius="0.01"/>
-            </geometry>
-        </collision>
-    </link>
-    <joint name="link1_to_hole1" type="fixed">
-        <parent link="link1"/>
-        <child link="hole1"/>
-        <origin xyz="0.04 0 0.01" rpy="0 0 0"/>
-    </joint>
-    <link name="hole8">
-        <inertial>
-            <origin xyz="0 0 0" rpy="0 0 0" />
-            <mass value="0.1" />
-            <inertia ixx="1E-9" ixy="0" ixz="0"
-                     iyy="1E-9" iyz="0"
-                     izz="1E-9" />
-        </inertial>
-        <visual>
-            <origin xyz="0 0 0" rpy="0 0 0"/>
-            <geometry>
-                <cylinder length="0.005" radius="0.01"/>
-            </geometry>
-            <material name="white" />
-        </visual>
-        <collision>
-            <origin xyz="0 0 0" rpy="0 0 0" />
-            <geometry>
-                <cylinder length="0.005" radius="0.01"/>
-            </geometry>
-        </collision>
-    </link>
-    <joint name="link1_to_hole8" type="fixed">
-        <parent link="link1"/>
-        <child link="hole8"/>
-        <origin xyz="0.02828 0.02828 0.01" rpy="0 0 0"/>
-    </joint>
-    <link name="hole7">
-        <inertial>
-            <origin xyz="0 0 0" rpy="0 0 0" />
-            <mass value="0.1" />
-            <inertia ixx="1E-9" ixy="0" ixz="0"
-                     iyy="1E-9" iyz="0"
-                     izz="1E-9" />
-        </inertial>
-        <visual>
-            <origin xyz="0 0 0" rpy="0 0 0"/>
-            <geometry>
-                <cylinder length="0.005" radius="0.01"/>
-            </geometry>
-            <material name="white" />
-        </visual>
-        <collision>
-            <origin xyz="0 0 0" rpy="0 0 0" />
-            <geometry>
-                <cylinder length="0.005" radius="0.01"/>
-            </geometry>
-        </collision>
-    </link>
-    <joint name="link1_to_hole7" type="fixed">
-        <parent link="link1"/>
-        <child link="hole7"/>
-        <origin xyz="0 0.04 0.01" rpy="0 0 0"/>
-    </joint>
-    <link name="hole6">
-        <inertial>
-            <origin xyz="0 0 0" rpy="0 0 0" />
-            <mass value="0.1" />
-            <inertia ixx="1E-9" ixy="0" ixz="0"
-                     iyy="1E-9" iyz="0"
-                     izz="1E-9" />
-        </inertial>
-        <visual>
-            <origin xyz="0 0 0" rpy="0 0 0"/>
-            <geometry>
-                <cylinder length="0.005" radius="0.01"/>
-            </geometry>
-            <material name="white" />
-        </visual>
-        <collision>
-            <origin xyz="0 0 0" rpy="0 0 0" />
-            <geometry>
-                <cylinder length="0.005" radius="0.01"/>
-            </geometry>
-        </collision>
-    </link>
-    <joint name="link1_to_hole6" type="fixed">
-        <parent link="link1"/>
-        <child link="hole6"/>
-        <origin xyz="-0.02828 0.02828 0.01" rpy="0 0 0"/>
-    </joint>
-    <link name="hole5">
-        <inertial>
-            <origin xyz="0 0 0" rpy="0 0 0" />
-            <mass value="0.1" />
-            <inertia ixx="1E-9" ixy="0" ixz="0"
-                     iyy="1E-9" iyz="0"
-                     izz="1E-9" />
-        </inertial>
-        <visual>
-            <origin xyz="0 0 0" rpy="0 0 0"/>
-            <geometry>
-                <cylinder length="0.005" radius="0.01"/>
-            </geometry>
-            <material name="white" />
-        </visual>
-        <collision>
-            <origin xyz="0 0 0" rpy="0 0 0" />
-            <geometry>
-                <cylinder length="0.005" radius="0.01"/>
-            </geometry>
-        </collision>
-    </link>
-    <joint name="link1_to_hole5" type="fixed">
-        <parent link="link1"/>
-        <child link="hole5"/>
-        <origin xyz="-0.04 0 0.01" rpy="0 0 0"/>
-    </joint>
-    <link name="hole4">
-        <inertial>
-            <origin xyz="0 0 0" rpy="0 0 0" />
-            <mass value="0.1" />
-            <inertia ixx="1E-9" ixy="0" ixz="0"
-                     iyy="1E-9" iyz="0"
-                     izz="1E-9" />
-        </inertial>
-        <visual>
-            <origin xyz="0 0 0" rpy="0 0 0"/>
-            <geometry>
-                <cylinder length="0.005" radius="0.01"/>
-            </geometry>
-            <material name="white" />
-        </visual>
-        <collision>
-            <origin xyz="0 0 0" rpy="0 0 0" />
-            <geometry>
-                <cylinder length="0.005" radius="0.01"/>
-            </geometry>
-        </collision>
-    </link>
-    <joint name="link1_to_hole4" type="fixed">
-        <parent link="link1"/>
-        <child link="hole4"/>
-        <origin xyz="-0.02828 -0.02828 0.01" rpy="0 0 0"/>
-    </joint>
-    <link name="hole3">
-        <inertial>
-            <origin xyz="0 0 0" rpy="0 0 0" />
-            <mass value="0.1" />
-            <inertia ixx="1E-9" ixy="0" ixz="0"
-                     iyy="1E-9" iyz="0"
-                     izz="1E-9" />
-        </inertial>
-        <visual>
-            <origin xyz="0 0 0" rpy="0 0 0"/>
-            <geometry>
-                <cylinder length="0.005" radius="0.01"/>
-            </geometry>
-            <material name="white" />
-        </visual>
-        <collision>
-            <origin xyz="0 0 0" rpy="0 0 0" />
-            <geometry>
-                <cylinder length="0.005" radius="0.01"/>
-            </geometry>
-        </collision>
-    </link>
-    <joint name="link1_to_hole3" type="fixed">
-        <parent link="link1"/>
-        <child link="hole3"/>
-        <origin xyz="0 -0.04 0.01" rpy="0 0 0"/>
-    </joint>
-    <link name="hole2">
-        <inertial>
-            <origin xyz="0 0 0" rpy="0 0 0" />
-            <mass value="0.1" />
-            <inertia ixx="1E-9" ixy="0" ixz="0"
-                     iyy="1E-9" iyz="0"
-                     izz="1E-9" />
-        </inertial>
-        <visual>
-            <origin xyz="0 0 0" rpy="0 0 0"/>
-            <geometry>
-                <cylinder length="0.005" radius="0.01"/>
-            </geometry>
-            <material name="white" />
-        </visual>
-        <collision>
-            <origin xyz="0 0 0" rpy="0 0 0" />
-            <geometry>
-                <cylinder length="0.005" radius="0.01"/>
-            </geometry>
-        </collision>
-    </link>
-    <joint name="link1_to_hole2" type="fixed">
-        <parent link="link1"/>
-        <child link="hole2"/>
-        <origin xyz="0.02828 -0.02828 0.01" rpy="0 0 0"/>
-    </joint>
+    <!--<link name="base">-->
+        <!--<inertial>-->
+            <!--<origin xyz="0 0 0" rpy="0 0 0" />-->
+            <!--<mass value="1" />-->
+            <!--<inertia ixx="1" ixy="0" ixz="0"-->
+                     <!--iyy="1" iyz="0"-->
+                     <!--izz="1" />-->
+        <!--</inertial>-->
+        <!--<visual>-->
+            <!--<origin xyz="0 0 0" rpy="0 0 0"/>-->
+            <!--<geometry>-->
+                <!--<box size="0.15 0.1 0.01"/>-->
+            <!--</geometry>-->
+            <!--<material name="sensoBlack" />-->
+        <!--</visual>-->
+        <!--&lt;!&ndash;<collision>&ndash;&gt;-->
+            <!--&lt;!&ndash;<origin xyz="0 0 0" rpy="0 0 0" />&ndash;&gt;-->
+            <!--&lt;!&ndash;<geometry>&ndash;&gt;-->
+                <!--&lt;!&ndash;<box size="0.15 0.1 0.01"/>&ndash;&gt;-->
+            <!--&lt;!&ndash;</geometry>&ndash;&gt;-->
+        <!--&lt;!&ndash;</collision>&ndash;&gt;-->
+    <!--</link>-->
+    <!--<joint name="world_to_base" type="fixed">-->
+        <!--<parent link="BaseBox"/>-->
+        <!--<child link="base"/>-->
+        <!--<origin xyz="0.40 0.15 0.005" rpy="0 0 ${90*DEG2RAD}" />-->
+        <!--<axis xyz="1 0 0" />-->
+    <!--</joint>-->
+    <!--<link name="base_link1">-->
+        <!--<inertial>-->
+            <!--<origin xyz="0 0 0" rpy="0 0 0" />-->
+            <!--<mass value="1" />-->
+            <!--<inertia ixx="1" ixy="0" ixz="0"-->
+                     <!--iyy="1" iyz="0"-->
+                     <!--izz="1" />-->
+        <!--</inertial>-->
+        <!--<visual>-->
+            <!--<origin xyz="0 0 0" rpy="0 0 0"/>-->
+            <!--<geometry>-->
+                <!--<cylinder length="0.01" radius="0.02"/>-->
+            <!--</geometry>-->
+            <!--<material name="sensoSilver" />-->
+        <!--</visual>-->
+        <!--&lt;!&ndash;<collision>&ndash;&gt;-->
+            <!--&lt;!&ndash;<origin xyz="0 0 0" rpy="0 0 0" />&ndash;&gt;-->
+            <!--&lt;!&ndash;<geometry>&ndash;&gt;-->
+                <!--&lt;!&ndash;<cylinder length="0.01" radius="0.02"/>&ndash;&gt;-->
+            <!--&lt;!&ndash;</geometry>&ndash;&gt;-->
+        <!--&lt;!&ndash;</collision>&ndash;&gt;-->
+    <!--</link>-->
+    <!--<joint name="base_to_base_link1" type="fixed">-->
+        <!--<parent link="base"/>-->
+        <!--<child link="base_link1"/>-->
+        <!--<origin xyz="0.05 0 0.01" rpy="0 0 0"/>-->
+        <!--<axis xyz="0 0 1" />-->
+    <!--</joint>-->
+    <!--<link name="link1">-->
+        <!--<inertial>-->
+            <!--<origin xyz="0 0 0" rpy="0 0 0" />-->
+            <!--<mass value="1" />-->
+            <!--<inertia ixx="1" ixy="0" ixz="0"-->
+                     <!--iyy="1" iyz="0"-->
+                     <!--izz="1" />-->
+        <!--</inertial>-->
+        <!--<visual>-->
+            <!--<origin xyz="0 0 0" rpy="0 0 0"/>-->
+            <!--<geometry>-->
+                <!--<cylinder length="0.01" radius="0.06"/>-->
+            <!--</geometry>-->
+            <!--<material name="sensoSilver" />-->
+        <!--</visual>-->
+        <!--&lt;!&ndash;<collision>&ndash;&gt;-->
+            <!--&lt;!&ndash;<origin xyz="0 0 0" rpy="0 0 0" />&ndash;&gt;-->
+            <!--&lt;!&ndash;<geometry>&ndash;&gt;-->
+                <!--&lt;!&ndash;<cylinder length="0.01" radius="0.06"/>&ndash;&gt;-->
+            <!--&lt;!&ndash;</geometry>&ndash;&gt;-->
+        <!--&lt;!&ndash;</collision>&ndash;&gt;-->
+    <!--</link>-->
+    <!--<joint name="base_link1_to_link1" type="revolute"> &lt;!&ndash; rotary table joint&ndash;&gt;-->
+        <!--<parent link="base_link1"/>-->
+        <!--<child link="link1"/>-->
+        <!--<origin xyz="0 0 0.01" rpy="0 0 0"/>-->
+        <!--<axis xyz="0 0 1" />-->
+        <!--<limit effort="1000" lower="0" upper="6.29" velocity="0"/>-->
+    <!--</joint>-->
+    <!--<link name="hole1">-->
+        <!--<inertial>-->
+            <!--<origin xyz="0 0 0" rpy="0 0 0" />-->
+            <!--<mass value="0.1" />-->
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