Commit message: SCARA and RT co-work in Moveit -succesful

File: gazebo_scara_and_rt/scara_v2_full_description/urdf/rotary_table_v2_urdf.xacro (robot description, xacro)
@@ -96,5 +96,5 @@
         <origin xyz="0 0 0.015" rpy="0 0 0"/>
         <axis xyz="0 0 1" />
-        <limit effort="1000" lower="-3.14" upper="3.14" velocity="0"/>
+        <limit effort="1000" lower="0" upper="6.29" velocity="0"/>
     </joint>
     <link name="hole1">
@@ -111,5 +111,5 @@
                 <cylinder length="0.005" radius="0.01"/>
             </geometry>
-            <material name="white" />
+            <material name="blue" />
         </visual>
         <collision>

File: gazebo_scara_and_rt/scara_v2_full_description/urdf/scara_and_rt_urdf.xacro (robot description, xacro)
@@ -444,9 +444,10 @@
         </collision>
     </link>
-    <joint name="base_link1_to_link1" type="continuous">
+    <joint name="base_link1_to_link1" type="revolute">
         <parent link="base_link1"/>
         <child link="link1"/>
         <origin xyz="0 0 0.01" rpy="0 0 0"/>
         <axis xyz="0 0 1" />
+        <limit effort="1000" lower="0" upper="6.29" velocity="0"/>
     </joint>
     <link name="hole1">
@@ -463,5 +464,5 @@
                 <cylinder length="0.005" radius="0.01"/>
             </geometry>
-            <material name="white" />
+            <material name="blue" />
         </visual>
         <collision>
@@ -859,16 +860,4 @@
     <!--</joint>-->
     <!--________________Transmision definitions______________________-->
-    <!--___rotary table___-->
-    <transmission name="RT_tran1">
-        <type>transmission_interface/SimpleTransmission</type>
-        <joint name="base_link1_to_link1">
-            <hardwareInterface>EffortJointInterface</hardwareInterface>
-        </joint>
-        <actuator name="RT_motor">
-            <hardwareInterface>EffortJointInterface</hardwareInterface>
-            <mechanicalReduction>1</mechanicalReduction>
-        </actuator>
-    </transmission>
-    <!--********************-->
     <!--___SCARA arm_____-->
     <transmission name="tran1">
@@ -893,3 +882,15 @@
     </transmission>
     <!--*******************-->
+    <!--___rotary table___-->
+    <transmission name="RT_tran1">
+        <type>transmission_interface/SimpleTransmission</type>
+        <joint name="base_link1_to_link1">
+            <hardwareInterface>EffortJointInterface</hardwareInterface>
+        </joint>
+        <actuator name="RT_motor">
+            <hardwareInterface>EffortJointInterface</hardwareInterface>
+            <mechanicalReduction>1</mechanicalReduction>
+        </actuator>
+    </transmission>
+    <!--********************-->
 </robot>

File: scara_v2_with_gripper/urdf/scara_and_rt_urdf.xacro (robot description, xacro)
@@ -483,5 +483,5 @@
                 <cylinder length="0.005" radius="0.01"/>
             </geometry>
-            <material name="white" />
+            <material name="blue" />
         </visual>
         <collision>

Commit message: SCARA and RT co-work in Moveit -full successful (with joint control)

File: gazebo_scara_and_rt/scara_v2_full_description/urdf/rotary_table_v2_urdf.xacro (robot description, xacro)
@@ -107,5 +107,5 @@
         </inertial>
         <visual>
-            <origin xyz="0.04 0 0" rpy="0 0 0"/>
+            <origin xyz="0 0 0" rpy="0 0 0"/>
             <geometry>
                 <cylinder length="0.005" radius="0.01"/>
@@ -123,5 +123,5 @@
         <parent link="link1"/>
         <child link="hole1"/>
-        <origin xyz="0 0 0.01" rpy="0 0 0"/>
+        <origin xyz="0.04 0 0.01" rpy="0 0 0"/>
     </joint>
     <link name="hole2">
@@ -134,5 +134,5 @@
         </inertial>
         <visual>
-            <origin xyz="0.02828 0.02828 0" rpy="0 0 0"/>
+            <origin xyz="0 0 0" rpy="0 0 0"/>
             <geometry>
                 <cylinder length="0.005" radius="0.01"/>
@@ -150,5 +150,5 @@
         <parent link="link1"/>
         <child link="hole2"/>
-        <origin xyz="0 0 0.01" rpy="0 0 0"/>
+        <origin xyz="0.02828 0.02828 0.01" rpy="0 0 0"/>
     </joint>
     <link name="hole3">
@@ -161,5 +161,5 @@
         </inertial>
         <visual>
-            <origin xyz="0 0.04 0" rpy="0 0 0"/>
+            <origin xyz="0 0 0" rpy="0 0 0"/>
             <geometry>
                 <cylinder length="0.005" radius="0.01"/>
@@ -177,5 +177,5 @@
         <parent link="link1"/>
         <child link="hole3"/>
-        <origin xyz="0 0 0.01" rpy="0 0 0"/>
+        <origin xyz="0 0.04 0.01" rpy="0 0 0"/>
     </joint>
     <link name="hole4">
@@ -188,5 +188,5 @@
         </inertial>
         <visual>
-            <origin xyz="-0.02828 0.02828 0" rpy="0 0 0"/>
+            <origin xyz="0 0 0" rpy="0 0 0"/>
             <geometry>
                 <cylinder length="0.005" radius="0.01"/>
@@ -204,5 +204,5 @@
         <parent link="link1"/>
         <child link="hole4"/>
-        <origin xyz="0 0 0.01" rpy="0 0 0"/>
+        <origin xyz="-0.02828 0.02828 0.01" rpy="0 0 0"/>
     </joint>
     <link name="hole5">
@@ -215,5 +215,5 @@
         </inertial>
         <visual>
-            <origin xyz="-0.04 0 0" rpy="0 0 0"/>
+            <origin xyz="0 0 0" rpy="0 0 0"/>
             <geometry>
                 <cylinder length="0.005" radius="0.01"/>
@@ -231,5 +231,5 @@
         <parent link="link1"/>
         <child link="hole5"/>
-        <origin xyz="0 0 0.01" rpy="0 0 0"/>
+        <origin xyz="-0.04 0 0.01" rpy="0 0 0"/>
     </joint>
     <link name="hole6">
@@ -242,5 +242,5 @@
         </inertial>
         <visual>
-            <origin xyz="-0.02828 -0.02828 0" rpy="0 0 0"/>
+            <origin xyz="0 0 0" rpy="0 0 0"/>
             <geometry>
                 <cylinder length="0.005" radius="0.01"/>
@@ -258,5 +258,5 @@
         <parent link="link1"/>
         <child link="hole6"/>
-        <origin xyz="0 0 0.01" rpy="0 0 0"/>
+        <origin xyz="-0.02828 -0.02828 0.01" rpy="0 0 0"/>
     </joint>
     <link name="hole7">
@@ -269,5 +269,5 @@
         </inertial>
         <visual>
-            <origin xyz="0 -0.04 0" rpy="0 0 0"/>
+            <origin xyz="0 0 0" rpy="0 0 0"/>
             <geometry>
                 <cylinder length="0.005" radius="0.01"/>
@@ -285,5 +285,5 @@
         <parent link="link1"/>
         <child link="hole7"/>
-        <origin xyz="0 0 0.01" rpy="0 0 0"/>
+        <origin xyz="0 -0.04 0.01" rpy="0 0 0"/>
     </joint>
     <link name="hole8">
@@ -296,5 +296,5 @@
         </inertial>
         <visual>
-            <origin xyz="0.02828 -0.02828 0" rpy="0 0 0"/>
+            <origin xyz="0 0 0" rpy="0 0 0"/>
             <geometry>
                 <cylinder length="0.005" radius="0.01"/>
@@ -312,5 +312,5 @@
         <parent link="link1"/>
         <child link="hole8"/>
-        <origin xyz="0 0 0.01" rpy="0 0 0"/>
+        <origin xyz="0.02828 -0.02828 0.01" rpy="0 0 0"/>
     </joint>
     <!--________________Transmision definitions______________________-->

File: gazebo_scara_and_rt/scara_v2_full_description/urdf/scara_and_rt_urdf.xacro (robot description, xacro)
@@ -460,5 +460,5 @@
         </inertial>
         <visual>
-            <origin xyz="0.04 0 0" rpy="0 0 0"/>
+            <origin xyz="0 0 0" rpy="0 0 0"/>
             <geometry>
                 <cylinder length="0.005" radius="0.01"/>
@@ -476,5 +476,5 @@
         <parent link="link1"/>
         <child link="hole1"/>
-        <origin xyz="0 0 0.0075" rpy="0 0 0"/>
+        <origin xyz="0.04 0 0.01" rpy="0 0 0"/>
     </joint>
     <link name="hole2">
@@ -487,5 +487,5 @@
         </inertial>
         <visual>
-            <origin xyz="0.02828 0.02828 0" rpy="0 0 0"/>
+            <origin xyz="0 0 0" rpy="0 0 0"/>
             <geometry>
                 <cylinder length="0.005" radius="0.01"/>
@@ -503,5 +503,5 @@
         <parent link="link1"/>
         <child link="hole2"/>
-        <origin xyz="0 0 0.0075" rpy="0 0 0"/>
+        <origin xyz="0.02828 0.02828 0.01" rpy="0 0 0"/>
     </joint>
     <link name="hole3">
@@ -514,5 +514,5 @@
         </inertial>
         <visual>
-            <origin xyz="0 0.04 0" rpy="0 0 0"/>
+            <origin xyz="0 0 0" rpy="0 0 0"/>
             <geometry>
                 <cylinder length="0.005" radius="0.01"/>
@@ -530,5 +530,5 @@
         <parent link="link1"/>
         <child link="hole3"/>
-        <origin xyz="0 0 0.0075" rpy="0 0 0"/>
+        <origin xyz="0 0.04 0.01" rpy="0 0 0"/>
     </joint>
     <link name="hole4">
@@ -541,5 +541,5 @@
         </inertial>
         <visual>
-            <origin xyz="-0.02828 0.02828 0" rpy="0 0 0"/>
+            <origin xyz="0 0 0" rpy="0 0 0"/>
             <geometry>
                 <cylinder length="0.005" radius="0.01"/>
@@ -557,5 +557,5 @@
         <parent link="link1"/>
         <child link="hole4"/>
-        <origin xyz="0 0 0.0075" rpy="0 0 0"/>
+        <origin xyz="-0.02828 0.02828 0.01" rpy="0 0 0"/>
     </joint>
     <link name="hole5">
@@ -568,5 +568,5 @@
         </inertial>
         <visual>
-            <origin xyz="-0.04 0 0" rpy="0 0 0"/>
+            <origin xyz="0 0 0" rpy="0 0 0"/>
             <geometry>
                 <cylinder length="0.005" radius="0.01"/>
@@ -584,5 +584,5 @@
         <parent link="link1"/>
         <child link="hole5"/>
-        <origin xyz="0 0 0.0075" rpy="0 0 0"/>
+        <origin xyz="-0.04 0 0.01" rpy="0 0 0"/>
     </joint>
     <link name="hole6">
@@ -595,5 +595,5 @@
         </inertial>
         <visual>
-            <origin xyz="-0.02828 -0.02828 0" rpy="0 0 0"/>
+            <origin xyz="0 0 0" rpy="0 0 0"/>
             <geometry>
                 <cylinder length="0.005" radius="0.01"/>
@@ -611,5 +611,5 @@
         <parent link="link1"/>
         <child link="hole6"/>
-        <origin xyz="0 0 0.0075" rpy="0 0 0"/>
+        <origin xyz="-0.02828 -0.02828 0.01" rpy="0 0 0"/>
     </joint>
     <link name="hole7">
@@ -622,5 +622,5 @@
         </inertial>
         <visual>
-            <origin xyz="0 -0.04 0" rpy="0 0 0"/>
+            <origin xyz="0 0 0" rpy="0 0 0"/>
             <geometry>
                 <cylinder length="0.005" radius="0.01"/>
@@ -638,5 +638,5 @@
         <parent link="link1"/>
         <child link="hole7"/>
-        <origin xyz="0 0 0.0075" rpy="0 0 0"/>
+        <origin xyz="0 -0.04 0.01" rpy="0 0 0"/>
     </joint>
     <link name="hole8">
@@ -649,5 +649,5 @@
         </inertial>
         <visual>
-            <origin xyz="0.02828 -0.02828 0" rpy="0 0 0"/>
+            <origin xyz="0 0 0" rpy="0 0 0"/>
             <geometry>
                 <cylinder length="0.005" radius="0.01"/>
@@ -665,5 +665,5 @@
         <parent link="link1"/>
         <child link="hole8"/>
-        <origin xyz="0 0 0.0075" rpy="0 0 0"/>
+        <origin xyz="0.02828 -0.02828 0.01" rpy="0 0 0"/>
     </joint>
     <!--*************************************-->

File: scara_v2_with_gripper/urdf/scara_and_rt_urdf.xacro (robot description, xacro)
@@ -178,5 +178,6 @@
         <parent link="placeBox" />
         <child link="placeHole1" />
-        <origin xyz="0.06 0.03 0.01" rpy="-3.8218E-18 -1.301E-16 -3.1416" />
+        <!--<origin xyz="0.06 0.03 0.01" rpy="-3.8218E-18 -1.301E-16 -3.1416" />-->
+        <origin xyz="-0.06 0.03 0.01" rpy="-3.8218E-18 -1.301E-16 -3.1416" />
         <axis xyz="1 0 0" />
     </joint>
@@ -207,5 +208,6 @@
         <parent link="placeBox" />
         <child link="placeHole2" />
-        <origin xyz="0.06 -0.03 0.01" rpy="-3.8218E-18 -1.301E-16 -3.1416" />
+        <!--<origin xyz="0.06 -0.03 0.01" rpy="-3.8218E-18 -1.301E-16 -3.1416" />-->
+        <origin xyz="-0.06 -0.03 0.01" rpy="-3.8218E-18 -1.301E-16 -3.1416" />
         <axis xyz="1 0 0" />
     </joint>
@@ -236,5 +238,6 @@
         <parent link="placeBox" />
         <child link="placeHole3" />
-        <origin xyz="0.02 0.03 0.01" rpy="-3.8218E-18 -1.301E-16 -3.1416" />
+        <!--<origin xyz="0.02 0.03 0.01" rpy="-3.8218E-18 -1.301E-16 -3.1416" />-->
+        <origin xyz="-0.02 0.03 0.01" rpy="-3.8218E-18 -1.301E-16 -3.1416" />
         <axis xyz="1 0 0" />
     </joint>
@@ -265,5 +268,6 @@
         <parent link="placeBox" />
         <child link="placeHole4" />
-        <origin xyz="0.02 -0.03 0.01" rpy="-3.8218E-18 -1.301E-16 -3.1416" />
+        <!--<origin xyz="0.02 -0.03 0.01" rpy="-3.8218E-18 -1.301E-16 -3.1416" />-->
+        <origin xyz="-0.02 -0.03 0.01" rpy="-3.8218E-18 -1.301E-16 -3.1416" />
         <axis xyz="1 0 0" />
     </joint>
@@ -294,5 +298,6 @@
         <parent link="placeBox" />
         <child link="placeHole5" />
-        <origin xyz="-0.02 0.03 0.01" rpy="-3.8218E-18 -1.301E-16 -3.1416" />
+        <!--<origin xyz="-0.02 0.03 0.01" rpy="-3.8218E-18 -1.301E-16 -3.1416" />-->
+        <origin xyz="0.02 0.03 0.01" rpy="-3.8218E-18 -1.301E-16 -3.1416" />
         <axis xyz="1 0 0" />
     </joint>
@@ -323,5 +328,6 @@
         <parent link="placeBox" />
         <child link="placeHole6" />
-        <origin xyz="-0.02 -0.03 0.01" rpy="-3.8218E-18 -1.301E-16 -3.1416" />
+        <!--<origin xyz="-0.02 -0.03 0.01" rpy="-3.8218E-18 -1.301E-16 -3.1416" />-->
+        <origin xyz="0.02 -0.03 0.01" rpy="-3.8218E-18 -1.301E-16 -3.1416" />
         <axis xyz="1 0 0" />
     </joint>
@@ -352,5 +358,6 @@
         <parent link="placeBox" />
         <child link="placeHole7" />
-        <origin xyz="-0.06 0.03 0.01" rpy="-3.8218E-18 -1.301E-16 -3.1416" />
+        <!--<origin xyz="-0.06 0.03 0.01" rpy="-3.8218E-18 -1.301E-16 -3.1416" />-->
+        <origin xyz="0.06 0.03 0.01" rpy="-3.8218E-18 -1.301E-16 -3.1416" />
         <axis xyz="1 0 0" />
     </joint>
@@ -381,5 +388,6 @@
         <parent link="placeBox" />
         <child link="placeHole8" />
-        <origin xyz="-0.06 -0.03 0.01" rpy="-3.8218E-18 -1.301E-16 -3.1416" />
+        <!--<origin xyz="-0.06 -0.03 0.01" rpy="-3.8218E-18 -1.301E-16 -3.1416" />-->
+        <origin xyz="0.06 -0.03 0.01" rpy="-3.8218E-18 -1.301E-16 -3.1416" />
         <axis xyz="1 0 0" />
     </joint>
@@ -464,9 +472,10 @@
         </collision>
     </link>
-    <joint name="base_link1_to_link1" type="continuous">
+    <joint name="base_link1_to_link1" type="revolute">
         <parent link="base_link1"/>
         <child link="link1"/>
         <origin xyz="0 0 0.01" rpy="0 0 0"/>
         <axis xyz="0 0 1" />
+        <limit effort="1000" lower="0" upper="6.29" velocity="0"/>
     </joint>
     <link name="hole1">
@@ -479,5 +488,5 @@
         </inertial>
         <visual>
-            <origin xyz="0.04 0 0" rpy="0 0 0"/>
+            <origin xyz="0 0 0" rpy="0 0 0"/>
             <geometry>
                 <cylinder length="0.005" radius="0.01"/>
@@ -495,7 +504,7 @@
         <parent link="link1"/>
         <child link="hole1"/>
-        <origin xyz="0 0 0.0075" rpy="0 0 0"/>
-    </joint>
-    <link name="hole2">
+        <origin xyz="0.04 0 0.01" rpy="0 0 0"/>
+    </joint>
+    <link name="hole8">
         <inertial>
             <origin xyz="0 0 0" rpy="0 0 0" />
@@ -506,5 +515,5 @@
         </inertial>
         <visual>
-            <origin xyz="0.02828 0.02828 0" rpy="0 0 0"/>
+            <origin xyz="0 0 0" rpy="0 0 0"/>
             <geometry>
                 <cylinder length="0.005" radius="0.01"/>
@@ -519,10 +528,10 @@
         </collision>
     </link>
-    <joint name="link1_to_hole2" type="fixed">
+    <joint name="link1_to_hole8" type="fixed">
         <parent link="link1"/>
-        <child link="hole2"/>
-        <origin xyz="0 0 0.0075" rpy="0 0 0"/>
-    </joint>
-    <link name="hole3">
+        <child link="hole8"/>
+        <origin xyz="0.02828 0.02828 0.01" rpy="0 0 0"/>
+    </joint>
+    <link name="hole7">
         <inertial>
             <origin xyz="0 0 0" rpy="0 0 0" />
@@ -533,5 +542,5 @@
         </inertial>
         <visual>
-            <origin xyz="0 0.04 0" rpy="0 0 0"/>
+            <origin xyz="0 0 0" rpy="0 0 0"/>
             <geometry>
                 <cylinder length="0.005" radius="0.01"/>
@@ -546,10 +555,10 @@
         </collision>
     </link>
-    <joint name="link1_to_hole3" type="fixed">
+    <joint name="link1_to_hole7" type="fixed">
         <parent link="link1"/>
-        <child link="hole3"/>
-        <origin xyz="0 0 0.0075" rpy="0 0 0"/>
-    </joint>
-    <link name="hole4">
+        <child link="hole7"/>
+        <origin xyz="0 0.04 0.01" rpy="0 0 0"/>
+    </joint>
+    <link name="hole6">
         <inertial>
             <origin xyz="0 0 0" rpy="0 0 0" />
@@ -560,5 +569,5 @@
         </inertial>
         <visual>
-            <origin xyz="-0.02828 0.02828 0" rpy="0 0 0"/>
+            <origin xyz="0 0 0" rpy="0 0 0"/>
             <geometry>
                 <cylinder length="0.005" radius="0.01"/>
@@ -573,8 +582,8 @@
         </collision>
     </link>
-    <joint name="link1_to_hole4" type="fixed">
+    <joint name="link1_to_hole6" type="fixed">
         <parent link="link1"/>
-        <child link="hole4"/>
-        <origin xyz="0 0 0.0075" rpy="0 0 0"/>
+        <child link="hole6"/>
+        <origin xyz="-0.02828 0.02828 0.01" rpy="0 0 0"/>
     </joint>
     <link name="hole5">
@@ -587,5 +596,5 @@
         </inertial>
         <visual>
-            <origin xyz="-0.04 0 0" rpy="0 0 0"/>
+            <origin xyz="0 0 0" rpy="0 0 0"/>
             <geometry>
                 <cylinder length="0.005" radius="0.01"/>
@@ -603,7 +612,7 @@
         <parent link="link1"/>
         <child link="hole5"/>
-        <origin xyz="0 0 0.0075" rpy="0 0 0"/>
-    </joint>
-    <link name="hole6">
+        <origin xyz="-0.04 0 0.01" rpy="0 0 0"/>
+    </joint>
+    <link name="hole4">
         <inertial>
             <origin xyz="0 0 0" rpy="0 0 0" />
@@ -614,5 +623,5 @@
         </inertial>
         <visual>
-            <origin xyz="-0.02828 -0.02828 0" rpy="0 0 0"/>
+            <origin xyz="0 0 0" rpy="0 0 0"/>
             <geometry>
                 <cylinder length="0.005" radius="0.01"/>
@@ -627,10 +636,10 @@
         </collision>
     </link>
-    <joint name="link1_to_hole6" type="fixed">
+    <joint name="link1_to_hole4" type="fixed">
         <parent link="link1"/>
-        <child link="hole6"/>
-        <origin xyz="0 0 0.0075" rpy="0 0 0"/>
-    </joint>
-    <link name="hole7">
+        <child link="hole4"/>
+        <origin xyz="-0.02828 -0.02828 0.01" rpy="0 0 0"/>
+    </joint>
+    <link name="hole3">
         <inertial>
             <origin xyz="0 0 0" rpy="0 0 0" />
@@ -641,5 +650,5 @@
         </inertial>
         <visual>
-            <origin xyz="0 -0.04 0" rpy="0 0 0"/>
+            <origin xyz="0 0 0" rpy="0 0 0"/>
             <geometry>
                 <cylinder length="0.005" radius="0.01"/>
@@ -654,10 +663,10 @@
         </collision>
     </link>
-    <joint name="link1_to_hole7" type="fixed">
+    <joint name="link1_to_hole3" type="fixed">
         <parent link="link1"/>
-        <child link="hole7"/>
-        <origin xyz="0 0 0.0075" rpy="0 0 0"/>
-    </joint>
-    <link name="hole8">
+        <child link="hole3"/>
+        <origin xyz="0 -0.04 0.01" rpy="0 0 0"/>
+    </joint>
+    <link name="hole2">
         <inertial>
             <origin xyz="0 0 0" rpy="0 0 0" />
@@ -668,5 +677,5 @@
         </inertial>
         <visual>
-            <origin xyz="0.02828 -0.02828 0" rpy="0 0 0"/>
+            <origin xyz="0 0 0" rpy="0 0 0"/>
             <geometry>
                 <cylinder length="0.005" radius="0.01"/>
@@ -681,8 +690,8 @@
         </collision>
     </link>
-    <joint name="link1_to_hole8" type="fixed">
+    <joint name="link1_to_hole2" type="fixed">
         <parent link="link1"/>
-        <child link="hole8"/>
-        <origin xyz="0 0 0.0075" rpy="0 0 0"/>
+        <child link="hole2"/>
+        <origin xyz="0.02828 -0.02828 0.01" rpy="0 0 0"/>
     </joint>
     <!--*************************************-->
