Commit message: dae bez cisla je SCARA s fake_jointom a dae1 je scara bez fake_jointu

File: gazebo_scara_and_rt/scara_v2_full_description/urdf/rotary_table_v2_urdf.xacro (robot description, xacro)
@@ -38,5 +38,5 @@
         <parent link="world"/>
         <child link="base"/>
-        <origin xyz="0 0 0" rpy="0 0 0" />
+        <origin xyz="0 0 0.01" rpy="0 0 0" />
         <axis xyz="1 0 0" />
     </joint>
@@ -96,5 +96,5 @@
         <origin xyz="0 0 0.015" rpy="0 0 0"/>
         <axis xyz="0 0 1" />
-        <limit effort="1000" lower="0" upper="6.29" velocity="0"/>
+        <limit effort="1000" lower="0" upper="6.29" velocity="10"/>
     </joint>
     <link name="hole1">
@@ -123,5 +123,5 @@
         <parent link="link1"/>
         <child link="hole1"/>
-        <origin xyz="0.04 0 0.01" rpy="0 0 0"/>
+        <origin xyz="0.04 0 0.0125" rpy="0 0 0"/>
     </joint>
     <link name="hole2">
@@ -150,5 +150,5 @@
         <parent link="link1"/>
         <child link="hole2"/>
-        <origin xyz="0.02828 0.02828 0.01" rpy="0 0 0"/>
+        <origin xyz="0.02828 0.02828 0.0125" rpy="0 0 0"/>
     </joint>
     <link name="hole3">
@@ -177,5 +177,5 @@
         <parent link="link1"/>
         <child link="hole3"/>
-        <origin xyz="0 0.04 0.01" rpy="0 0 0"/>
+        <origin xyz="0 0.04 0.0125" rpy="0 0 0"/>
     </joint>
     <link name="hole4">
@@ -204,5 +204,5 @@
         <parent link="link1"/>
         <child link="hole4"/>
-        <origin xyz="-0.02828 0.02828 0.01" rpy="0 0 0"/>
+        <origin xyz="-0.02828 0.02828 0.0125" rpy="0 0 0"/>
     </joint>
     <link name="hole5">
@@ -231,5 +231,5 @@
         <parent link="link1"/>
         <child link="hole5"/>
-        <origin xyz="-0.04 0 0.01" rpy="0 0 0"/>
+        <origin xyz="-0.04 0 0.0125" rpy="0 0 0"/>
     </joint>
     <link name="hole6">
@@ -258,5 +258,5 @@
         <parent link="link1"/>
         <child link="hole6"/>
-        <origin xyz="-0.02828 -0.02828 0.01" rpy="0 0 0"/>
+        <origin xyz="-0.02828 -0.02828 0.0125" rpy="0 0 0"/>
     </joint>
     <link name="hole7">
@@ -285,5 +285,5 @@
         <parent link="link1"/>
         <child link="hole7"/>
-        <origin xyz="0 -0.04 0.01" rpy="0 0 0"/>
+        <origin xyz="0 -0.04 0.0125" rpy="0 0 0"/>
     </joint>
     <link name="hole8">
@@ -312,8 +312,8 @@
         <parent link="link1"/>
         <child link="hole8"/>
-        <origin xyz="0.02828 -0.02828 0.01" rpy="0 0 0"/>
+        <origin xyz="0.02828 -0.02828 0.0125" rpy="0 0 0"/>
     </joint>
     <!--________________Transmision definitions______________________-->
-    <transmission name="RT_tran1">
+    <transmission name="tran1rt">
         <type>transmission_interface/SimpleTransmission</type>
         <joint name="base_link1_to_link1">

File: scara_v2_with_gripper/urdf/scara_v2_with_gripper_urdf.urdf (robot description, URDF)
Before this commit: robot scara_v2, 12 links, 11 joints
Joints:
- joint Joint2: origin xyz=0.24972  0 0.081 rpy=0 0 0 -> xyz=0.24972  0 0.081 rpy=0 0 1.57

File: scara_v2_with_gripper/urdf/scara_v2_with_gripper_urdf.xacro (robot description, xacro)
@@ -210,5 +210,5 @@
         <parent link="ScaraLink1" />
         <child link="ScaraLink2" />
-        <origin xyz="0.24972  0 0.081" rpy="0 0 0" />
+        <origin xyz="0.24972  0 0.081" rpy="0 0 1.57" />
         <axis xyz="0 0 1" />
         <!--<limit effort="0" lower="-2.65" upper="2.65" velocity="0"/>-->
@@ -218,13 +218,13 @@
     <!--     GRIPPER JOINTS DEFINITION    -->
     <!--Revolute joint for IKfast-->
-    <link name="fake_link"/>
-    <joint name="fake_joint" type="revolute">
-        <parent link="ScaraLink2" />
-        <child link="fake_link" />
-        <!--<origin xyz="0 -0.24305 0.0424 " rpy="0 0 3.1416" />-->
-        <origin xyz="0 -0.24305 -0.0424 " rpy="0 0 3.1416" />
-        <axis xyz="0 0 1" />
-        <limit effort="1000.0" lower="0.0" upper="0.001" velocity="0"/>
-    </joint>
+    <!--<link name="fake_link"/>-->
+    <!--<joint name="fake_joint" type="revolute">-->
+        <!--<parent link="ScaraLink2" />-->
+        <!--<child link="fake_link" />-->
+        <!--&lt;!&ndash;<origin xyz="0 -0.24305 0.0424 " rpy="0 0 3.1416" />&ndash;&gt;-->
+        <!--<origin xyz="0 -0.24305 -0.0424 " rpy="0 0 3.1416" />-->
+        <!--<axis xyz="0 0 1" />-->
+        <!--<limit effort="1000.0" lower="0.0" upper="0.001" velocity="0"/>-->
+    <!--</joint>-->
     <link name="GripperBase">
         <inertial>
@@ -251,8 +251,9 @@
     </link>
     <joint name="Joint_GripperBase" type="prismatic">
-        <parent link="fake_link" />
+        <!--<parent link="fake_link" />-->
+        <parent link="ScaraLink2" />
         <child link="GripperBase" />
-        <origin xyz="0 0 0" rpy="0 0 0" />
-        <!--<origin xyz="0 -0.0424 0.24305" rpy="3.1416 0 3.1416" />-->
+        <!--<origin xyz="0 0 0" rpy="0 0 0" />-->
+        <origin xyz="0 -0.24305 -0.0424 " rpy="0 0 3.1416" />
         <axis xyz="0 0 1" />
         <limit effort="1000.0" lower="-0.04" upper="0.05" velocity="1"/>

Commit message: Gazebo SCARA, RT, SCARA_and_RT - everything works!
Signed-off-by: dluhosko@gmail.com <dluhosko>

File: gazebo_scara_and_rt/scara_v2_full_description/urdf/rotary_table_v2_urdf.xacro (robot description, xacro)
@@ -4,4 +4,5 @@
     <xacro:property name="DEG2RAD" value="0.01745329252" />
     <xacro:property name="RED2DEG" value="57.295779513" />
+    <xacro:property name="M_PI" value="3.141592" />
     <!-- ***********************************  -->
     <!-- Import all Gazebo-customization elements, including Gazebo colors -->
@@ -96,5 +97,5 @@
         <origin xyz="0 0 0.015" rpy="0 0 0"/>
         <axis xyz="0 0 1" />
-        <limit effort="1000" lower="0" upper="6.29" velocity="10"/>
+        <limit effort="100" lower="0" upper="${2*M_PI}" velocity="0.5"/>
     </joint>
     <link name="hole1">

File: gazebo_scara_and_rt/scara_v2_full_description/urdf/scara_and_rt_urdf.xacro (robot description, xacro)
@@ -4,4 +4,5 @@
     <xacro:property name="DEG2RAD" value="0.01745329252" />
     <xacro:property name="RED2DEG" value="57.295779513" />
+    <xacro:property name="M_PI" value="3.141592" />
     <!-- ***********************************  -->
     <!-- Import all Gazebo-customization elements, including Gazebo colors -->
@@ -456,5 +457,5 @@
         <origin xyz="0 0 0.01" rpy="0 0 0"/>
         <axis xyz="0 0 1" />
-        <limit effort="1000" lower="0" upper="6.29" velocity="0"/>
+        <limit effort="100" lower="0" upper="${2*M_PI}" velocity="0.5"/>
     </joint>
     <link name="hole1">
@@ -734,5 +735,5 @@
         <axis xyz="0 1 0" />
         <!--<limit effort="0" lower="-1.57079" upper="1.57079" velocity="0"/>-->
-        <limit effort="0" lower="${-85*DEG2RAD}" upper="${85*DEG2RAD}" velocity="0"/>
+        <limit effort="100" lower="${-85*DEG2RAD}" upper="${85*DEG2RAD}" velocity="2"/>
     </joint>
     <link name="ScaraLink2">
@@ -765,5 +766,5 @@
         <axis xyz="0 1 0" />
         <!--<limit effort="0" lower="-2.65" upper="2.65" velocity="0"/>-->
-        <limit effort="0" lower="${-170*DEG2RAD}" upper="${170*DEG2RAD}" velocity="0"/>
+        <limit effort="100" lower="${-170*DEG2RAD}" upper="${170*DEG2RAD}" velocity="2"/>
     </joint>
     <!--**********************************-->
@@ -871,8 +872,8 @@
         <type>transmission_interface/SimpleTransmission</type>
         <joint name="Joint1">
-            <hardwareInterface>EffortJointInterface</hardwareInterface>
+            <hardwareInterface>hardware_interface/EffortJointInterface</hardwareInterface>
         </joint>
         <actuator name="motor1">
-            <hardwareInterface>EffortJointInterface</hardwareInterface>
+            <hardwareInterface>hardware_interface/EffortJointInterface</hardwareInterface>
             <mechanicalReduction>1</mechanicalReduction>
         </actuator>
@@ -881,8 +882,8 @@
         <type>transmission_interface/SimpleTransmission</type>
         <joint name="Joint2">
-            <hardwareInterface>EffortJointInterface</hardwareInterface>
+            <hardwareInterface>hardware_interface/EffortJointInterface</hardwareInterface>
         </joint>
         <actuator name="motor2">
-            <hardwareInterface>EffortJointInterface</hardwareInterface>
+            <hardwareInterface>hardware_interface/EffortJointInterface</hardwareInterface>
             <mechanicalReduction>1</mechanicalReduction>
         </actuator>
@@ -893,9 +894,9 @@
         <type>transmission_interface/SimpleTransmission</type>
         <joint name="base_link1_to_link1">
-            <hardwareInterface>EffortJointInterface</hardwareInterface>
+            <hardwareInterface>hardware_interface/EffortJointInterface</hardwareInterface>
         </joint>
         <actuator name="RT_motor">
-            <hardwareInterface>EffortJointInterface</hardwareInterface>
-            <mechanicalReduction>1</mechanicalReduction>
+            <hardwareInterface>hardware_interface/EffortJointInterface</hardwareInterface>
+            <mechanicalReduction>100000</mechanicalReduction>
         </actuator>
     </transmission>
