Commit message: SCARA and RT co-work in Moveit -full successful (with joint control)

File: gazebo_scara_and_rt/scara_v2_full_description/urdf/scara_and_rt_urdf.xacro (robot description, xacro)
@@ -9,5 +9,4 @@
     <!-- ****************************************************************  -->
     <!--        Import Material colors        -->
-    <!--Z nejakeho dovodu mi nechce nacitat materials.........-->
     <xacro:include filename="$(find scara_v2_full_description)/urdf/materials.xacro" />
     <!-- Link and Joint definitions  -->
@@ -158,5 +157,6 @@
         <parent link="placeBox" />
         <child link="placeHole1" />
-        <origin xyz="0.06 0.03 0.01" rpy="-3.8218E-18 -1.301E-16 -3.1416" />
+        <!--<origin xyz="0.06 0.03 0.01" rpy="-3.8218E-18 -1.301E-16 -3.1416" />-->
+        <origin xyz="-0.06 0.03 0.01" rpy="-3.8218E-18 -1.301E-16 -3.1416" />
         <axis xyz="1 0 0" />
     </joint>
@@ -187,5 +187,6 @@
         <parent link="placeBox" />
         <child link="placeHole2" />
-        <origin xyz="0.06 -0.03 0.01" rpy="-3.8218E-18 -1.301E-16 -3.1416" />
+        <!--<origin xyz="0.06 -0.03 0.01" rpy="-3.8218E-18 -1.301E-16 -3.1416" />-->
+        <origin xyz="-0.06 -0.03 0.01" rpy="-3.8218E-18 -1.301E-16 -3.1416" />
         <axis xyz="1 0 0" />
     </joint>
@@ -216,5 +217,6 @@
         <parent link="placeBox" />
         <child link="placeHole3" />
-        <origin xyz="0.02 0.03 0.01" rpy="-3.8218E-18 -1.301E-16 -3.1416" />
+        <!--<origin xyz="0.02 0.03 0.01" rpy="-3.8218E-18 -1.301E-16 -3.1416" />-->
+        <origin xyz="-0.02 0.03 0.01" rpy="-3.8218E-18 -1.301E-16 -3.1416" />
         <axis xyz="1 0 0" />
     </joint>
@@ -245,5 +247,6 @@
         <parent link="placeBox" />
         <child link="placeHole4" />
-        <origin xyz="0.02 -0.03 0.01" rpy="-3.8218E-18 -1.301E-16 -3.1416" />
+        <!--<origin xyz="0.02 -0.03 0.01" rpy="-3.8218E-18 -1.301E-16 -3.1416" />-->
+        <origin xyz="-0.02 -0.03 0.01" rpy="-3.8218E-18 -1.301E-16 -3.1416" />
         <axis xyz="1 0 0" />
     </joint>
@@ -274,5 +277,6 @@
         <parent link="placeBox" />
         <child link="placeHole5" />
-        <origin xyz="-0.02 0.03 0.01" rpy="-3.8218E-18 -1.301E-16 -3.1416" />
+        <!--<origin xyz="-0.02 0.03 0.01" rpy="-3.8218E-18 -1.301E-16 -3.1416" />-->
+        <origin xyz="0.02 0.03 0.01" rpy="-3.8218E-18 -1.301E-16 -3.1416" />
         <axis xyz="1 0 0" />
     </joint>
@@ -303,5 +307,6 @@
         <parent link="placeBox" />
         <child link="placeHole6" />
-        <origin xyz="-0.02 -0.03 0.01" rpy="-3.8218E-18 -1.301E-16 -3.1416" />
+        <!--<origin xyz="-0.02 -0.03 0.01" rpy="-3.8218E-18 -1.301E-16 -3.1416" />-->
+        <origin xyz="0.02 -0.03 0.01" rpy="-3.8218E-18 -1.301E-16 -3.1416" />
         <axis xyz="1 0 0" />
     </joint>
@@ -332,5 +337,6 @@
         <parent link="placeBox" />
         <child link="placeHole7" />
-        <origin xyz="-0.06 0.03 0.01" rpy="-3.8218E-18 -1.301E-16 -3.1416" />
+        <!--<origin xyz="-0.06 0.03 0.01" rpy="-3.8218E-18 -1.301E-16 -3.1416" />-->
+        <origin xyz="0.06 0.03 0.01" rpy="-3.8218E-18 -1.301E-16 -3.1416" />
         <axis xyz="1 0 0" />
     </joint>
@@ -361,5 +367,6 @@
         <parent link="placeBox" />
         <child link="placeHole8" />
-        <origin xyz="-0.06 -0.03 0.01" rpy="-3.8218E-18 -1.301E-16 -3.1416" />
+        <!--<origin xyz="-0.06 -0.03 0.01" rpy="-3.8218E-18 -1.301E-16 -3.1416" />-->
+        <origin xyz="0.06 -0.03 0.01" rpy="-3.8218E-18 -1.301E-16 -3.1416" />
         <axis xyz="1 0 0" />
     </joint>

Commit message: rotary table fixed, controllers fixed

File: gazebo_scara_and_rt/scara_v2_full_description/urdf/scara_and_rt_urdf.xacro (robot description, xacro)
@@ -4,4 +4,5 @@
     <xacro:property name="DEG2RAD" value="0.01745329252" />
     <xacro:property name="RED2DEG" value="57.295779513" />
+    <xacro:property name="M_PI" value="3.141592" />
     <!-- ***********************************  -->
     <!-- Import all Gazebo-customization elements, including Gazebo colors -->
@@ -456,5 +457,5 @@
         <origin xyz="0 0 0.01" rpy="0 0 0"/>
         <axis xyz="0 0 1" />
-        <limit effort="1000" lower="0" upper="6.29" velocity="0"/>
+        <limit effort="100" lower="0" upper="${2*M_PI}" velocity="0.5"/>
     </joint>
     <link name="hole1">
@@ -734,5 +735,5 @@
         <axis xyz="0 1 0" />
         <!--<limit effort="0" lower="-1.57079" upper="1.57079" velocity="0"/>-->
-        <limit effort="0" lower="${-85*DEG2RAD}" upper="${85*DEG2RAD}" velocity="0"/>
+        <limit effort="100" lower="${-85*DEG2RAD}" upper="${85*DEG2RAD}" velocity="100"/>
     </joint>
     <link name="ScaraLink2">
@@ -765,5 +766,5 @@
         <axis xyz="0 1 0" />
         <!--<limit effort="0" lower="-2.65" upper="2.65" velocity="0"/>-->
-        <limit effort="0" lower="${-170*DEG2RAD}" upper="${170*DEG2RAD}" velocity="0"/>
+        <limit effort="100" lower="${-170*DEG2RAD}" upper="${170*DEG2RAD}" velocity="100"/>
     </joint>
     <!--**********************************-->
@@ -871,8 +872,8 @@
         <type>transmission_interface/SimpleTransmission</type>
         <joint name="Joint1">
-            <hardwareInterface>EffortJointInterface</hardwareInterface>
+            <hardwareInterface>hardware_interface/EffortJointInterface</hardwareInterface>
         </joint>
         <actuator name="motor1">
-            <hardwareInterface>EffortJointInterface</hardwareInterface>
+            <hardwareInterface>hardware_interface/EffortJointInterface</hardwareInterface>
             <mechanicalReduction>1</mechanicalReduction>
         </actuator>
@@ -881,8 +882,8 @@
         <type>transmission_interface/SimpleTransmission</type>
         <joint name="Joint2">
-            <hardwareInterface>EffortJointInterface</hardwareInterface>
+            <hardwareInterface>hardware_interface/EffortJointInterface</hardwareInterface>
         </joint>
         <actuator name="motor2">
-            <hardwareInterface>EffortJointInterface</hardwareInterface>
+            <hardwareInterface>hardware_interface/EffortJointInterface</hardwareInterface>
             <mechanicalReduction>1</mechanicalReduction>
         </actuator>
@@ -893,9 +894,9 @@
         <type>transmission_interface/SimpleTransmission</type>
         <joint name="base_link1_to_link1">
-            <hardwareInterface>EffortJointInterface</hardwareInterface>
+            <hardwareInterface>hardware_interface/EffortJointInterface</hardwareInterface>
         </joint>
         <actuator name="RT_motor">
-            <hardwareInterface>EffortJointInterface</hardwareInterface>
-            <mechanicalReduction>1</mechanicalReduction>
+            <hardwareInterface>hardware_interface/EffortJointInterface</hardwareInterface>
+            <mechanicalReduction>100000</mechanicalReduction>
         </actuator>
     </transmission>

Commit message: Gazebo SCARA, RT, SCARA_and_RT - everything works!
Signed-off-by: dluhosko@gmail.com <dluhosko>

File: gazebo_scara_and_rt/scara_v2_full_description/urdf/scara_and_rt_urdf.xacro (robot description, xacro)
@@ -770,34 +770,34 @@
     <!--**********************************-->
     <!--     GRIPPER JOINTS DEFINITION    -->
-    <!--<link name="GripperBase">-->
-        <!--<inertial>-->
-            <!--<origin xyz="0 0 0" rpy="0 0 0" />-->
-            <!--<mass  value="1" />-->
-            <!--<inertia  ixx="1E-6" ixy="0" ixz="0"-->
-                      <!--iyy="1E-6" iyz="0"-->
-                      <!--izz="1E-6" />-->
-        <!--</inertial>-->
-        <!--<visual>-->
-            <!--<origin  xyz="0 0 0"  rpy="0 0 0" />-->
-            <!--<geometry>-->
-                <!--<mesh filename="package://scara_v2_with_gripper/meshes/GripperBase.STL" />-->
-            <!--</geometry>-->
-            <!--<material name="sensoDarkGray">-->
-            <!--</material>-->
-        <!--</visual>-->
-        <!--<collision>-->
-            <!--<origin xyz="0 0 0" rpy="0 0 0" />-->
-            <!--<geometry>-->
-                <!--<mesh filename="package://scara_v2_with_gripper/meshes/GripperBase.STL" />-->
-            <!--</geometry>-->
-        <!--</collision>-->
-    <!--</link>-->
-    <!--<joint name="Joint_GripperBase" type="prismatic">-->
-        <!--<parent link="ScaraLink2" />-->
-        <!--<child link="GripperBase" />-->
-        <!--<origin xyz="0 -0.0424 0.24305" rpy="3.1416 0 3.1416" />-->
-        <!--<axis xyz="0 1 0" />-->
-        <!--<limit effort="1000.0" lower="-0.04" upper="0.05" velocity="1"/>-->
-    <!--</joint>-->
+    <link name="GripperBase">
+        <inertial>
+            <origin xyz="0 0 0" rpy="0 0 0" />
+            <mass  value="0.5" />
+            <inertia  ixx="0.01" ixy="0.01" ixz="0.01"
+                      iyy="0.01" iyz="0.01"
+                      izz="0.01" />
+        </inertial>
+        <visual>
+            <origin  xyz="0 0 0"  rpy="0 0 0" />
+            <geometry>
+                <mesh filename="package://scara_v2_with_gripper/meshes/GripperBase.STL" />
+            </geometry>
+            <material name="sensoDarkGray">
+            </material>
+        </visual>
+        <collision>
+            <origin xyz="0 0 0" rpy="0 0 0" />
+            <geometry>
+                <mesh filename="package://scara_v2_with_gripper/meshes/GripperBase.STL" />
+            </geometry>
+        </collision>
+    </link>
+    <joint name="Joint_GripperBase" type="prismatic">
+        <parent link="ScaraLink2" />
+        <child link="GripperBase" />
+        <origin xyz="0 -0.0424 0.24305" rpy="3.1416 0 3.1416" />
+        <axis xyz="0 1 0" />
+        <limit effort="100.0" lower="-0.04" upper="0.05" velocity="1"/>
+    </joint>
     <!--<joint name="Base_to_tool0" type="fixed">-->
         <!--<parent link="GripperBase" />-->
@@ -889,4 +889,14 @@
         </actuator>
     </transmission>
+    <transmission name="tran3">
+        <type>transmission_interface/SimpleTransmission</type>
+        <joint name="Joint_GripperBase">
+            <hardwareInterface>EffortJointInterface</hardwareInterface>
+        </joint>
+        <actuator name="motor3">
+            <hardwareInterface>EffortJointInterface</hardwareInterface>
+            <mechanicalReduction>100</mechanicalReduction>
+        </actuator>
+    </transmission>
     <!--*******************-->
     <!--___rotary table___-->

File: gazebo_scara_and_rt/scara_v2_full_description/urdf/scara_v2_urdf.xacro (robot description, xacro)
@@ -456,34 +456,35 @@
     <!--**********************************-->
     <!--     GRIPPER JOINTS DEFINITION    -->
-     <!--<link name="GripperBase">-->
-         <!--<inertial>-->
-             <!--<origin xyz="0 0 0" rpy="0 0 0" />-->
-             <!--<mass  value="1" />-->
-             <!--<inertia  ixx="1E-6" ixy="0" ixz="0"-->
-                     <!--iyy="1E-6" iyz="0"-->
-                     <!--izz="1E-6" />-->
-         <!--</inertial>-->
-         <!--<visual>-->
-             <!--<origin  xyz="0 0 0"  rpy="0 0 0" />-->
-             <!--<geometry>-->
-                 <!--<mesh filename="package://scara_v2_with_gripper/meshes/GripperBase.STL" />-->
-             <!--</geometry>-->
-             <!--<material name="sensoDarkGray">-->
-             <!--</material>-->
-         <!--</visual>-->
-         <!--<collision>-->
-             <!--<origin xyz="0 0 0" rpy="0 0 0" />-->
-             <!--<geometry>-->
-                 <!--<mesh filename="package://scara_v2_with_gripper/meshes/GripperBase.STL" />-->
-             <!--</geometry>-->
-         <!--</collision>-->
-     <!--</link>-->
-     <!--<joint name="Joint_GripperBase" type="prismatic">-->
-         <!--<parent link="ScaraLink2" />-->
-         <!--<child link="GripperBase" />-->
-         <!--<origin xyz="0 -0.0424 0.24305" rpy="3.1416 0 3.1416" />-->
-         <!--<axis xyz="0 1 0" />-->
-         <!--<limit effort="1000.0" lower="-0.04" upper="0.05" velocity="1"/>-->
-     <!--</joint>-->
+     <link name="GripperBase">
+         <inertial>
+             <origin xyz="0 0 0" rpy="0 0 0" />
+             <mass  value="1" />
+             <inertia  ixx="1E-6" ixy="0" ixz="0"
+                     iyy="1E-6" iyz="0"
+                     izz="1E-6" />
+         </inertial>
+         <visual>
+             <origin  xyz="0 0 0"  rpy="0 0 0" />
+             <geometry>
+                 <mesh filename="package://scara_v2_with_gripper/meshes/GripperBase.STL" />
+             </geometry>
+             <material name="sensoDarkGray">
+             </material>
+         </visual>
+         <collision>
+             <origin xyz="0 0 0" rpy="0 0 0" />
+             <geometry>
+                 <mesh filename="package://scara_v2_with_gripper/meshes/GripperBase.STL" />
+             </geometry>
+         </collision>
+     </link>
+     <joint name="Joint_GripperBase" type="prismatic">
+         <parent link="ScaraLink2" />
+         <child link="GripperBase" />
+         <origin xyz="0 -0.0424 0.24305" rpy="3.1416 0 3.1416" />
+         <axis xyz="0 1 0" />
+         <limit effort="100" lower="-0.04" upper="0.05" velocity="1.0"/>
+         <dynamics damping="50" friction="1"/>
+     </joint>
      <!--<link name="GripperLeft">-->
          <!--<inertial>-->
@@ -567,4 +568,5 @@
         <actuator name="motor2">
             <hardwareInterface>EffortJointInterface</hardwareInterface>
+            <!--EffortJointInterface-->
             <mechanicalReduction>1</mechanicalReduction>
         </actuator>
@@ -572,14 +574,14 @@
     <!--*******************-->
     <!--_____Gripper_______-->
-    <!--<transmission name="tran3">-->
-        <!--<type>transmission_interface/SimpleTransmission</type>-->
-        <!--<joint name="Joint_GripperBase">-->
-            <!--<hardwareInterface>PositionJointInterface</hardwareInterface>-->
-        <!--</joint>-->
-        <!--<actuator name="motor3">-->
-            <!--<hardwareInterface>PositionJointInterface</hardwareInterface>-->
-            <!--<mechanicalReduction>1</mechanicalReduction>-->
-        <!--</actuator>-->
-    <!--</transmission>-->
+    <transmission name="tran3">
+        <type>transmission_interface/SimpleTransmission</type>
+        <joint name="Joint_GripperBase">
+            <hardwareInterface>EffortJointInterface</hardwareInterface>
+        </joint>
+        <actuator name="motor3">
+            <hardwareInterface>EffortJointInterface</hardwareInterface>
+            <mechanicalReduction>100</mechanicalReduction>
+        </actuator>
+    </transmission>
     <!--<transmission name="tran4">-->
         <!--<type>transmission_interface/SimpleTransmission</type>-->

Commit message: Gazebo gripper control from topic enabled
Signed-off-by: dluhosko@gmail.com <dluhosko>

File: gazebo_scara_and_rt/scara_v2_full_description/urdf/scara_and_rt_urdf.xacro (robot description, xacro)
@@ -735,5 +735,5 @@
         <axis xyz="0 1 0" />
         <!--<limit effort="0" lower="-1.57079" upper="1.57079" velocity="0"/>-->
-        <limit effort="100" lower="${-85*DEG2RAD}" upper="${85*DEG2RAD}" velocity="100"/>
+        <limit effort="20" lower="${-85*DEG2RAD}" upper="${85*DEG2RAD}" velocity="100"/>        <!--100-->
     </joint>
     <link name="ScaraLink2">
@@ -766,5 +766,5 @@
         <axis xyz="0 1 0" />
         <!--<limit effort="0" lower="-2.65" upper="2.65" velocity="0"/>-->
-        <limit effort="100" lower="${-170*DEG2RAD}" upper="${170*DEG2RAD}" velocity="100"/>
+        <limit effort="20" lower="${-170*DEG2RAD}" upper="${170*DEG2RAD}" velocity="100"/><!--100-->
     </joint>
     <!--**********************************-->
@@ -806,65 +806,65 @@
     <!--</joint>-->
     <!--<link name="tool0"/>-->
-    <!--<link name="GripperLeft">-->
-        <!--<inertial>-->
-            <!--<origin  xyz="0 0 0"  rpy="3.14 0 0" />-->
-            <!--<mass value="1" />-->
-            <!--<inertia ixx="1E-6"  ixy="0" ixz="0"-->
-                     <!--iyy="1E-6" iyz="0"-->
-                     <!--izz="1E-6" />-->
-        <!--</inertial>-->
-        <!--<visual>-->
-            <!--<origin xyz="0 0 0" rpy="3.14 0 0" />-->
-            <!--<geometry>-->
-                <!--<mesh filename="package://scara_v2_with_gripper/meshes/gripperLeft_full.STL" />-->
-            <!--</geometry>-->
-            <!--<material name="sensoDarkGray">-->
-            <!--</material>-->
-        <!--</visual>-->
-        <!--<collision>-->
-            <!--<origin xyz="0 0 0" rpy="3.14 0 0" />-->
-            <!--<geometry>-->
-                <!--<mesh  filename="package://scara_v2_with_gripper/meshes/gripperLeft_full.STL" />-->
-            <!--</geometry>-->
-        <!--</collision>-->
-    <!--</link>-->
-    <!--<joint name="Joint_Gripper" type="prismatic">-->
-        <!--<parent link="GripperBase" />-->
-        <!--<child link="GripperLeft" />-->
-        <!--<origin xyz="-0.0162 0.0984 0" rpy="3.1416 0 0" />-->
-        <!--<axis xyz="1 0 0" />-->
-        <!--<limit effort="1000.0" lower="0" upper="0.003" velocity="1"/>-->
-    <!--</joint>-->
-    <!--<link name="GripperRight">-->
-        <!--<inertial>-->
-            <!--<origin   xyz="0 0 0" rpy="3.14 0 0" />-->
-            <!--<mass value="1" />-->
-            <!--<inertia  ixx="1E-6"  ixy="0" ixz="0"-->
-                      <!--iyy="1E-6" iyz="0"-->
-                      <!--izz="1E-6" />-->
-        <!--</inertial>-->
-        <!--<visual>-->
-            <!--<origin  xyz="0 0 0"  rpy="3.14 0 0" />-->
-            <!--<geometry>-->
-                <!--<mesh filename="package://scara_v2_with_gripper/meshes/gripperRight_full.STL" />-->
-            <!--</geometry>-->
-            <!--<material name="sensoDarkGray">-->
-            <!--</material>-->
-        <!--</visual>-->
-        <!--<collision>-->
-            <!--<origin  xyz="0 0 0" rpy="3.14 0 0" />-->
-            <!--<geometry>-->
-                <!--<mesh  filename="package://scara_v2_with_gripper/meshes/gripperRight_full.STL" />-->
-            <!--</geometry>-->
-        <!--</collision>-->
-    <!--</link>-->
-    <!--<joint name="Joint_GripperRight" type="prismatic">-->
-        <!--<parent link="GripperBase" />-->
-        <!--<child link="GripperRight" />-->
-        <!--<origin  xyz="0.0165 0.0984 0" rpy="3.1416 0 3.1416" />-->
-        <!--<axis  xyz="1 0 0" />-->
-        <!--<limit effort="1000.0" lower="0" upper="0.003" velocity="1"/>-->
+    <link name="GripperLeft">
+        <inertial>
+            <origin  xyz="0 0 0"  rpy="3.14 0 0" />
+            <mass value="0.1" />
+            <inertia  ixx="0.01" ixy="0.01" ixz="0.01"
+                      iyy="0.01" iyz="0.01"
+                      izz="0.01" />
+        </inertial>
+        <visual>
+            <origin xyz="0 0 0" rpy="3.14 0 0" />
+            <geometry>
+                <mesh filename="package://scara_v2_with_gripper/meshes/gripperLeft_full.STL" />
+            </geometry>
+            <material name="sensoDarkGray">
+            </material>
+        </visual>
+        <collision>
+            <origin xyz="0 0 0" rpy="3.14 0 0" />
+            <geometry>
+                <mesh  filename="package://scara_v2_with_gripper/meshes/gripperLeft_full.STL" />
+            </geometry>
+        </collision>
+    </link>
+    <joint name="Joint_Gripper" type="prismatic">
+        <parent link="GripperBase" />
+        <child link="GripperLeft" />
+        <origin xyz="-0.0162 0.0984 0" rpy="3.1416 0 0" />
+        <axis xyz="1 0 0" />
+        <limit effort="100.0" lower="0" upper="0.003" velocity="1"/>
+    </joint>
+    <link name="GripperRight">
+        <inertial>
+            <origin   xyz="0 0 0" rpy="3.14 0 0" />
+            <mass value="0.1" />
+            <inertia  ixx="0.01" ixy="0.01" ixz="0.01"
+                      iyy="0.01" iyz="0.01"
+                      izz="0.01" />
+        </inertial>
+        <visual>
+            <origin  xyz="0 0 0"  rpy="3.14 0 0" />
+            <geometry>
+                <mesh filename="package://scara_v2_with_gripper/meshes/gripperRight_full.STL" />
+            </geometry>
+            <material name="sensoDarkGray">
+            </material>
+        </visual>
+        <collision>
+            <origin  xyz="0 0 0" rpy="3.14 0 0" />
+            <geometry>
+                <mesh  filename="package://scara_v2_with_gripper/meshes/gripperRight_full.STL" />
+            </geometry>
+        </collision>
+    </link>
+    <joint name="Joint_GripperRight" type="prismatic">
+        <parent link="GripperBase" />
+        <child link="GripperRight" />
+        <origin  xyz="0.0165 0.0984 0" rpy="3.1416 0 3.1416" />
+        <axis  xyz="1 0 0" />
+        <limit effort="1000.0" lower="0" upper="0.003" velocity="1"/>
         <!--<mimic joint="Joint_Gripper" multiplier="1" offset="0" />-->
-    <!--</joint>-->
+    </joint>
     <!--________________Transmision definitions______________________-->
     <!--___SCARA arm_____-->
@@ -900,4 +900,26 @@
     </transmission>
     <!--*******************-->
+    <!--_____Gripper_______-->
+    <transmission name="tran4">
+        <type>transmission_interface/SimpleTransmission</type>
+        <joint name="Joint_Gripper">
+            <hardwareInterface>EffortJointInterface</hardwareInterface>
+        </joint>
+        <actuator name="motor4">
+            <hardwareInterface>EffortJointInterface</hardwareInterface>
+            <mechanicalReduction>100</mechanicalReduction>
+        </actuator>
+    </transmission>
+    <transmission name="tran5">
+        <type>transmission_interface/SimpleTransmission</type>
+        <joint name="Joint_GripperRight">
+            <hardwareInterface>EffortJointInterface</hardwareInterface>
+        </joint>
+        <actuator name="motor5">
+            <hardwareInterface>EffortJointInterface</hardwareInterface>
+            <mechanicalReduction>100</mechanicalReduction>
+        </actuator>
+    </transmission>
+    <!-- ***************************** -->
     <!--___rotary table___-->
     <transmission name="RT_tran1">
@@ -908,5 +930,5 @@
         <actuator name="RT_motor">
             <hardwareInterface>hardware_interface/EffortJointInterface</hardwareInterface>
-            <mechanicalReduction>100000</mechanicalReduction>
+            <mechanicalReduction>1000</mechanicalReduction>
         </actuator>
     </transmission>

File: gazebo_scara_and_rt/scara_v2_full_description/urdf/scara_v2_urdf.xacro (robot description, xacro)
@@ -459,8 +459,8 @@
          <inertial>
              <origin xyz="0 0 0" rpy="0 0 0" />
-             <mass  value="1" />
-             <inertia  ixx="1E-6" ixy="0" ixz="0"
-                     iyy="1E-6" iyz="0"
-                     izz="1E-6" />
+             <mass  value="0.5" />
+             <inertia  ixx="0.01" ixy="0.01" ixz="0.01"
+                       iyy="0.01" iyz="0.01"
+                       izz="0.01" />
          </inertial>
          <visual>
