Commit message: matlab-moveit comunication

File: gazebo_scara_and_rt/scara_v2_full_description/urdf/scara_and_rt_urdf.xacro (robot description, xacro)
@@ -122,5 +122,5 @@
             <origin xyz="0 0 0" rpy="0 0 0" />
             <geometry>
-                <box size="0.2 0.15 0.02"/>
+                <box size="0.2 0.12 0.02"/>
             </geometry>
         </collision>
@@ -392,5 +392,5 @@
             <origin xyz="0 0 0" rpy="0 0 0" />
             <geometry>
-                <box size="0.15 0.1 0.02"/>
+                <box size="0.15 0.1 0.01"/>
             </geometry>
         </collision>
@@ -448,5 +448,5 @@
             <origin xyz="0 0 0" rpy="0 0 0" />
             <geometry>
-                <cylinder length="0.02" radius="0.06"/>
+                <cylinder length="0.01" radius="0.06"/>
             </geometry>
         </collision>
@@ -801,7 +801,7 @@
     </joint>
     <!--<joint name="Base_to_tool0" type="fixed">-->
-        <!--<parent link="GripperBase" />-->
-        <!--<child link="tool0" />-->
-        <!--<origin xyz="0 0.0984 0" rpy="0 0 0 " />-->
+    <!--<parent link="GripperBase" />-->
+    <!--<child link="tool0" />-->
+    <!--<origin xyz="0 0.0984 0" rpy="0 0 0 " />-->
     <!--</joint>-->
     <!--<link name="tool0"/>-->
@@ -829,10 +829,10 @@
         </collision>
     </link>
-    <joint name="Joint_Gripper" type="prismatic">
+    <joint name="Joint_Gripper" type="fixed">
         <parent link="GripperBase" />
         <child link="GripperLeft" />
         <origin xyz="-0.0162 0.0984 0" rpy="3.1416 0 0" />
         <axis xyz="1 0 0" />
-        <limit effort="100.0" lower="0" upper="0.003" velocity="1"/>
+        <!--<limit effort="100.0" lower="0" upper="0.003" velocity="1"/>-->
     </joint>
     <link name="GripperRight">
@@ -859,10 +859,10 @@
         </collision>
     </link>
-    <joint name="Joint_GripperRight" type="prismatic">
+    <joint name="Joint_GripperRight" type="fixed">
         <parent link="GripperBase" />
         <child link="GripperRight" />
         <origin  xyz="0.0165 0.0984 0" rpy="3.1416 0 3.1416" />
         <axis  xyz="1 0 0" />
-        <limit effort="1000.0" lower="0" upper="0.003" velocity="1"/>
+        <!--<limit effort="1000.0" lower="0" upper="0.003" velocity="1"/>-->
         <!--<mimic joint="Joint_Gripper" multiplier="1" offset="0" />-->
     </joint>
@@ -901,24 +901,24 @@
     <!--*******************-->
     <!--_____Gripper_______-->
-    <transmission name="tran4">
-        <type>transmission_interface/SimpleTransmission</type>
-        <joint name="Joint_Gripper">
-            <hardwareInterface>EffortJointInterface</hardwareInterface>
-        </joint>
-        <actuator name="motor4">
-            <hardwareInterface>EffortJointInterface</hardwareInterface>
-            <mechanicalReduction>100</mechanicalReduction>
-        </actuator>
-    </transmission>
-    <transmission name="tran5">
-        <type>transmission_interface/SimpleTransmission</type>
-        <joint name="Joint_GripperRight">
-            <hardwareInterface>EffortJointInterface</hardwareInterface>
-        </joint>
-        <actuator name="motor5">
-            <hardwareInterface>EffortJointInterface</hardwareInterface>
-            <mechanicalReduction>100</mechanicalReduction>
-        </actuator>
-    </transmission>
+    <!--<transmission name="tran4">-->
+    <!--<type>transmission_interface/SimpleTransmission</type>-->
+    <!--<joint name="Joint_Gripper">-->
+    <!--<hardwareInterface>EffortJointInterface</hardwareInterface>-->
+    <!--</joint>-->
+    <!--<actuator name="motor4">-->
+    <!--<hardwareInterface>EffortJointInterface</hardwareInterface>-->
+    <!--<mechanicalReduction>100</mechanicalReduction>-->
+    <!--</actuator>-->
+    <!--</transmission>-->
+    <!--<transmission name="tran5">-->
+    <!--<type>transmission_interface/SimpleTransmission</type>-->
+    <!--<joint name="Joint_GripperRight">-->
+    <!--<hardwareInterface>EffortJointInterface</hardwareInterface>-->
+    <!--</joint>-->
+    <!--<actuator name="motor5">-->
+    <!--<hardwareInterface>EffortJointInterface</hardwareInterface>-->
+    <!--<mechanicalReduction>100</mechanicalReduction>-->
+    <!--</actuator>-->
+    <!--</transmission>-->
     <!-- ***************************** -->
     <!--___rotary table___-->

File: gazebo_scara_and_rt/scara_v2_full_description/urdf/scara_v2_urdf.xacro (robot description, xacro)
@@ -2,4 +2,7 @@
 <robot  name="scara_v2_full" xmlns:xacro="http://www.ros.org/wiki/xacro">
     <!--              Constants               -->
+    <xacro:property name="DEG2RAD" value="0.01745329252" />
+    <xacro:property name="RED2DEG" value="57.295779513" />
+    <xacro:property name="M_PI" value="3.141592" />
     <!-- ***********************************  -->
     <!-- Import all Gazebo-customization elements, including Gazebo colors -->
@@ -368,7 +371,7 @@
             <origin xyz="0 0 0" rpy="0 0 0" />
             <mass value="1" />
-            <inertia ixx="0.01" ixy="0.01" ixz="0.01"
-                     iyy="0.01" iyz="0.01"
-                     izz="0.01" />
+            <inertia ixx="1" ixy="0" ixz="0"
+                     iyy="1" iyz="0"
+                     izz="1" />
         </inertial>
         <visual>
@@ -387,10 +390,9 @@
         </collision>
     </link>
-    <joint name="Joint_ScaraBase" type="revolute">
+    <joint name="Joint_ScaraBase" type="fixed">
         <parent link="BaseBox" />
         <child link="ScaraBase" />
         <origin xyz="0.212 0.58 0.141"  rpy="1.5708 0 0" />
         <axis  xyz="1 0 0" />
-        <limit effort="0" lower="0" upper="0" velocity="0"/>
     </joint>
     <link name="ScaraLink1">
@@ -405,5 +407,5 @@
             <origin xyz="0 0 0" rpy="0 0 0" />
             <geometry>
-                <mesh filename="package://scara_v2_with_gripper/meshes/ScaraLink1.STL" />
+                <mesh filename="package://scara_v2_with_gripper/meshes/ScaraLink1.STL" />   <!--ScaraLink1.STL-->
             </geometry>
             <material name="sensoSilver">
@@ -422,5 +424,6 @@
         <origin xyz="0 0.051 0" rpy="0 0 0" />
         <axis xyz="0 1 0" />
-        <limit effort="1000" lower="-1.57079" upper="1.57079" velocity="0"/>
+        <!--<limit effort="0" lower="-1.57079" upper="1.57079" velocity="0"/>-->
+        <limit effort="20" lower="${-85*DEG2RAD}" upper="${85*DEG2RAD}" velocity="100"/>        <!--100-->
     </joint>
     <link name="ScaraLink2">
@@ -429,6 +432,6 @@
             <mass value="1.5020" />
             <inertia  ixx="5.0471E-2" ixy="3.0689E-4" ixz="-8.5622E-4"
-                    iyy="4.7456E-2" iyz="8.7643E-3"
-                    izz="5.2228E-3" />
+                      iyy="4.7456E-2" iyz="8.7643E-3"
+                      izz="5.2228E-3" />
         </inertial>
         <visual>
@@ -452,101 +455,107 @@
         <origin xyz="0.24972 -0.081 0" rpy="3.14 -1.5708 0" />
         <axis xyz="0 1 0" />
-        <limit effort="1000" lower="-2.65" upper="2.65" velocity="0"/>
+        <!--<limit effort="0" lower="-2.65" upper="2.65" velocity="0"/>-->
+        <limit effort="20" lower="${-170*DEG2RAD}" upper="${170*DEG2RAD}" velocity="100"/><!--100-->
     </joint>
     <!--**********************************-->
     <!--     GRIPPER JOINTS DEFINITION    -->
-     <link name="GripperBase">
-         <inertial>
-             <origin xyz="0 0 0" rpy="0 0 0" />
-             <mass  value="0.5" />
-             <inertia  ixx="0.01" ixy="0.01" ixz="0.01"
-                       iyy="0.01" iyz="0.01"
-                       izz="0.01" />
-         </inertial>
-         <visual>
-             <origin  xyz="0 0 0"  rpy="0 0 0" />
-             <geometry>
-                 <mesh filename="package://scara_v2_with_gripper/meshes/GripperBase.STL" />
-             </geometry>
-             <material name="sensoDarkGray">
-             </material>
-         </visual>
-         <collision>
-             <origin xyz="0 0 0" rpy="0 0 0" />
-             <geometry>
-                 <mesh filename="package://scara_v2_with_gripper/meshes/GripperBase.STL" />
-             </geometry>
-         </collision>
-     </link>
-     <joint name="Joint_GripperBase" type="prismatic">
-         <parent link="ScaraLink2" />
-         <child link="GripperBase" />
-         <origin xyz="0 -0.0424 0.24305" rpy="3.1416 0 3.1416" />
-         <axis xyz="0 1 0" />
-         <limit effort="100" lower="-0.04" upper="0.05" velocity="1.0"/>
-         <dynamics damping="50" friction="1"/>
-     </joint>
-     <!--<link name="GripperLeft">-->
-         <!--<inertial>-->
-             <!--<origin  xyz="0 0 0"  rpy="3.14 0 0" />-->
-             <!--<mass value="1" />-->
-             <!--<inertia ixx="1E-6"  ixy="0" ixz="0"-->
-                     <!--iyy="1E-6" iyz="0"-->
-                     <!--izz="1E-6" />-->
-         <!--</inertial>-->
-         <!--<visual>-->
-             <!--<origin xyz="0 0 0" rpy="3.14 0 0" />-->
-             <!--<geometry>-->
-                 <!--<mesh filename="package://scara_v2_with_gripper/meshes/gripperLeft_full.STL" />-->
-             <!--</geometry>-->
-             <!--<material name="sensoDarkGray">-->
-             <!--</material>-->
-         <!--</visual>-->
-         <!--<collision>-->
-             <!--<origin xyz="0 0 0" rpy="0 0 0" />-->
-             <!--<geometry>-->
-                 <!--<mesh  filename="package://scara_v2_with_gripper/meshes/gripperLeft_full.STL" />-->
-             <!--</geometry>-->
-         <!--</collision>-->
-     <!--</link>-->
-     <!--<joint name="Joint_Gripper" type="prismatic">-->
-         <!--<parent link="GripperBase" />-->
-         <!--<child link="GripperLeft" />-->
-         <!--<origin xyz="-0.0162 0.0984 0" rpy="3.1416 0 0" />-->
-         <!--<axis xyz="1 0 0" />-->
-         <!--<limit effort="1000.0" lower="0" upper="0.003" velocity="1"/>-->
-     <!--</joint>-->
-     <!--<link name="GripperRight">-->
-         <!--<inertial>-->
-             <!--<origin   xyz="0 0 0" rpy="3.14 0 0" />-->
-             <!--<mass value="1" />-->
-             <!--<inertia  ixx="1E-6"  ixy="0" ixz="0"-->
-                     <!--iyy="1E-6" iyz="0"-->
-                     <!--izz="1E-6" />-->
-         <!--</inertial>-->
-         <!--<visual>-->
-             <!--<origin  xyz="0 0 0"  rpy="3.14 0 0" />-->
-             <!--<geometry>-->
-                 <!--<mesh filename="package://scara_v2_with_gripper/meshes/gripperRight_full.STL" />-->
-             <!--</geometry>-->
-             <!--<material name="sensoDarkGray">-->
-             <!--</material>-->
-         <!--</visual>-->
-         <!--<collision>-->
-             <!--<origin  xyz="0 0 0" rpy="0 0 0" />-->
-             <!--<geometry>-->
-                 <!--<mesh  filename="package://scara_v2_with_gripper/meshes/gripperRight_full.STL" />-->
-             <!--</geometry>-->
-         <!--</collision>-->
-     <!--</link>-->
-     <!--<joint name="Joint_GripperRight" type="prismatic">-->
-         <!--<parent link="GripperBase" />-->
-         <!--<child link="GripperRight" />-->
-         <!--<origin  xyz="0.0165 0.0984 0" rpy="3.1416 0 3.1416" />-->
-         <!--<axis  xyz="1 0 0" />-->
-         <!--<limit effort="1000.0" lower="-0.003" upper="0.003" velocity="1"/>-->
-         <!--<mimic joint="Joint_Gripper" multiplier="1" offset="0" />-->
-     <!--</joint>-->
-     <!---->
+    <link name="GripperBase">
+        <inertial>
+            <origin xyz="0 0 0" rpy="0 0 0" />
+            <mass  value="0.5" />
+            <inertia  ixx="0.01" ixy="0.01" ixz="0.01"
+                      iyy="0.01" iyz="0.01"
+                      izz="0.01" />
+        </inertial>
+        <visual>
+            <origin  xyz="0 0 0"  rpy="0 0 0" />
+            <geometry>
+                <mesh filename="package://scara_v2_with_gripper/meshes/GripperBase.STL" />
+            </geometry>
+            <material name="sensoDarkGray">
+            </material>
+        </visual>
+        <collision>
+            <origin xyz="0 0 0" rpy="0 0 0" />
+            <geometry>
+                <mesh filename="package://scara_v2_with_gripper/meshes/GripperBase.STL" />
+            </geometry>
+        </collision>
+    </link>
+    <joint name="Joint_GripperBase" type="prismatic">
+        <parent link="ScaraLink2" />
+        <child link="GripperBase" />
+        <origin xyz="0 -0.0424 0.24305" rpy="3.1416 0 3.1416" />
+        <axis xyz="0 1 0" />
+        <limit effort="100.0" lower="-0.04" upper="0.05" velocity="1"/>
+    </joint>
+    <!--<joint name="Base_to_tool0" type="fixed">-->
+    <!--<parent link="GripperBase" />-->
+    <!--<child link="tool0" />-->
+    <!--<origin xyz="0 0.0984 0" rpy="0 0 0 " />-->
+    <!--</joint>-->
+    <!--<link name="tool0"/>-->
+    <link name="GripperLeft">
+        <inertial>
+            <origin  xyz="0 0 0"  rpy="3.14 0 0" />
+            <mass value="0.05" />
+            <inertia  ixx="0.001" ixy="0.001" ixz="0.001"
+                      iyy="0.001" iyz="0.001"
+                      izz="0.001" />
+            </inertial>
+        <visual>
+            <origin xyz="0 0 0" rpy="3.14 0 0" />
+            <geometry>
+                <mesh filename="package://scara_v2_with_gripper/meshes/gripperLeft_full.STL" />
+            </geometry>
+            <material name="sensoDarkGray">
+            </material>
+        </visual>
+        <collision>
+            <origin xyz="0 0 0" rpy="3.14 0 0" />
+            <geometry>
+                <mesh  filename="package://scara_v2_with_gripper/meshes/gripperLeft_full.STL" />
+            </geometry>
+        </collision>
+    </link>
+    <joint name="Joint_Gripper" type="prismatic">
+        <parent link="GripperBase" />
+        <child link="GripperLeft" />
+        <origin xyz="-0.0162 0.0984 0" rpy="3.1416 0 0" />
+        <axis xyz="1 0 0" />
+        <limit effort="100.0" lower="0" upper="0.003" velocity="1"/>
+    </joint>
+    <link name="GripperRight">
+        <inertial>
+            <origin  xyz="0 0 0"  rpy="3.14 0 0" />
+            <mass value="0.05" />
+            <inertia  ixx="0.001" ixy="0.001" ixz="0.001"
+                      iyy="0.001" iyz="0.001"
+                      izz="0.001" />
+        </inertial>
+        <visual>
+            <origin  xyz="0 0 0"  rpy="3.14 0 0" />
+            <geometry>
+                <mesh filename="package://scara_v2_with_gripper/meshes/gripperRight_full.STL" />
+            </geometry>
+            <material name="sensoDarkGray">
+            </material>
+        </visual>
+        <collision>
+            <origin  xyz="0 0 0" rpy="3.14 0 0" />
+            <geometry>
+                <mesh  filename="package://scara_v2_with_gripper/meshes/gripperRight_full.STL" />
+            </geometry>
+        </collision>
+    </link>
+    <joint name="Joint_GripperRight" type="fixed">
+        <parent link="GripperBase" />
+        <child link="GripperRight" />
+        <origin  xyz="0.0165 0.0984 0" rpy="3.1416 0 3.1416" />
+        <!--<origin  xyz="0.1 0.0984 0" rpy="3.1416 0 3.1416" />-->
+        <axis  xyz="1 0 0" />
+        <limit effort="100.0" lower="0" upper="0.003" velocity="1"/>
+        <!--<mimic joint="Joint_Gripper" multiplier="1" offset="0" />-->
+    </joint>
      <!--________________Transmision definitions______________________-->
     <!--___SCARA arm_____-->
@@ -584,13 +593,24 @@
         </actuator>
     </transmission>
-    <!--<transmission name="tran4">-->
-        <!--<type>transmission_interface/SimpleTransmission</type>-->
-        <!--<joint name="Joint_Gripper">-->
-            <!--<hardwareInterface>EffortJointInterface</hardwareInterface>-->
-        <!--</joint>-->
-        <!--<actuator name="motor4">-->
-            <!--<hardwareInterface>EffortJointInterface</hardwareInterface>-->
-            <!--<mechanicalReduction>1000</mechanicalReduction>-->
-        <!--</actuator>-->
+    <!--gripper pick and place-->
+    <transmission name="tran4">
+    <type>transmission_interface/SimpleTransmission</type>
+    <joint name="Joint_Gripper">
+    <hardwareInterface>EffortJointInterface</hardwareInterface>
+    </joint>
+    <actuator name="motor4">
+    <hardwareInterface>EffortJointInterface</hardwareInterface>
+    <mechanicalReduction>1</mechanicalReduction>
+    </actuator>
+    </transmission>
+    <!--<transmission name="tran5">-->
+    <!--<type>transmission_interface/SimpleTransmission</type>-->
+    <!--<joint name="Joint_GripperRight">-->
+    <!--<hardwareInterface>EffortJointInterface</hardwareInterface>-->
+    <!--</joint>-->
+    <!--<actuator name="motor5">-->
+    <!--<hardwareInterface>EffortJointInterface</hardwareInterface>-->
+    <!--<mechanicalReduction>100</mechanicalReduction>-->
+    <!--</actuator>-->
     <!--</transmission>-->
     <!-- ***************************** -->
