Commit message: matlab-moveit comunication

File: scara_v2_with_gripper/urdf/rotary_table_v2_urdf.xacro (robot description, xacro)
@@ -1,37 +1,18 @@
 <?xml version="1.0"?>
 <robot  name="rotary_table_v2" xmlns:xacro="http://www.ros.org/wiki/xacro">
-    <!--  Material Color definitions -->
-    <material name="white">
-        <color rgba="1 1 1 1"/>
-    </material>
-    <material name="blue">
-        <color rgba="0 0 1 1"/>
-    </material>
-    <material name="red">
-        <color rgba="1 0 0 1"/>
-    </material>
-    <material name="green">
-        <color rgba="0 1 0 1"/>
-    </material>
-    <material name="sensoSilver">
-        <color rgba="0.839216 0.839216 0.839216 1"/>
-    </material>
-    <material name="sensoBlack">
-        <color rgba="0 0 0 1 "/>
-    </material>
-    <material name="sensoGray">
-        <color rgba="0.466667 0.533333 0.6 1 "/>
-    </material>
-    <material name="sensoDarkGray">
-        <color rgba="0.156863 0.156863 0.156863 1 "/>
-    </material>
-    <!--****************************-->
-    <!--**********MACROS************-->
+    <!--              Constants               -->
     <xacro:property name="DEG2RAD" value="0.01745329252" />
     <xacro:property name="RED2DEG" value="57.295779513" />
-    <!--****************************-->
-    <!-- Link and Joint definitions  -->
+    <xacro:property name="M_PI" value="3.141592" />
+    <!-- ***********************************  -->
+    <!-- Import all Gazebo-customization elements, including Gazebo colors -->
+    <xacro:include filename="$(find scara_v2_full_description)/urdf/rotary_table_v2_gazebo.gazebo" />
+    <!-- ****************************************************************  -->
+    <!--        Import Material colors        -->
+    <xacro:include filename="$(find scara_v2_full_description)/urdf/materials.xacro" />
+    <!-- ***********************************  -->
     <link name="world"/>
-    <link name="base">
+    <!--Casual box-->
+    <link name="casualBox">
         <inertial>
             <origin xyz="0 0 0" rpy="0 0 0" />
@@ -44,6 +25,35 @@
             <origin xyz="0 0 0" rpy="0 0 0"/>
             <geometry>
+                <box size="0.5 0.5 0.5"/>
+            </geometry>
+            <material name="white" />
+        </visual>
+        <collision>
+            <origin xyz="0 0 0" rpy="0 0 0" />
+            <geometry>
                 <box size="0.15 0.1 0.02"/>
             </geometry>
+        </collision>
+    </link>
+    <joint name="world_to_casualBox" type="fixed">
+        <parent link="world"/>
+        <child link="casualBox"/>
+        <origin xyz="0 0 0.25" rpy="0 0 0" />
+        <axis xyz="1 0 0" />
+    </joint>
+    <!-- Link and Joint definitions  -->
+    <link name="base">
+        <inertial>
+            <origin xyz="0 0 0" rpy="0 0 0" />
+            <mass value="1" />
+            <inertia ixx="1" ixy="0" ixz="0"
+                     iyy="1" iyz="0"
+                     izz="1" />
+        </inertial>
+        <visual>
+            <origin xyz="0 0 0" rpy="0 0 0"/>
+            <geometry>
+                <box size="0.15 0.1 0.02"/>
+            </geometry>
             <material name="sensoBlack" />
         </visual>
@@ -56,7 +66,7 @@
     </link>
     <joint name="world_to_base" type="fixed">
-        <parent link="world"/>
+        <parent link="casualBox"/>
         <child link="base"/>
-        <origin xyz="0 0 0" rpy="0 0 0" />
+        <origin xyz="0 0 0.26" rpy="0 0 0" />
         <axis xyz="1 0 0" />
     </joint>
@@ -111,9 +121,10 @@
         </collision>
     </link>
-    <joint name="base_link1_to_link1" type="continuous">
+    <joint name="rotary_table_joint" type="revolute">    <!-- joint name base_link1_to_link1-->
         <parent link="base_link1"/>
         <child link="link1"/>
         <origin xyz="0 0 0.015" rpy="0 0 0"/>
         <axis xyz="0 0 1" />
+        <limit effort="100" lower="0" upper="${2*M_PI}" velocity="0.5"/>
     </joint>
     <link name="hole1">
@@ -126,9 +137,9 @@
         </inertial>
         <visual>
-            <origin xyz="0.04 0 0" rpy="0 0 0"/>
-            <geometry>
-                <cylinder length="0.005" radius="0.01"/>
-            </geometry>
-            <material name="white" />
+            <origin xyz="0 0 0" rpy="0 0 0"/>
+            <geometry>
+                <cylinder length="0.005" radius="0.01"/>
+            </geometry>
+            <material name="blue" />
         </visual>
         <collision>
@@ -142,5 +153,5 @@
         <parent link="link1"/>
         <child link="hole1"/>
-        <origin xyz="0 0 0.01" rpy="0 0 0"/>
+        <origin xyz="0.04 0 0.0125" rpy="0 0 0"/>
     </joint>
     <link name="hole2">
@@ -153,5 +164,5 @@
         </inertial>
         <visual>
-            <origin xyz="0.02828 0.02828 0" rpy="0 0 0"/>
+            <origin xyz="0 0 0" rpy="0 0 0"/>
             <geometry>
                 <cylinder length="0.005" radius="0.01"/>
@@ -169,5 +180,5 @@
         <parent link="link1"/>
         <child link="hole2"/>
-        <origin xyz="0 0 0.01" rpy="0 0 0"/>
+        <origin xyz="0.02828 0.02828 0.0125" rpy="0 0 0"/>
     </joint>
     <link name="hole3">
@@ -180,5 +191,5 @@
         </inertial>
         <visual>
-            <origin xyz="0 0.04 0" rpy="0 0 0"/>
+            <origin xyz="0 0 0" rpy="0 0 0"/>
             <geometry>
                 <cylinder length="0.005" radius="0.01"/>
@@ -196,5 +207,5 @@
         <parent link="link1"/>
         <child link="hole3"/>
-        <origin xyz="0 0 0.01" rpy="0 0 0"/>
+        <origin xyz="0 0.04 0.0125" rpy="0 0 0"/>
     </joint>
     <link name="hole4">
@@ -207,5 +218,5 @@
         </inertial>
         <visual>
-            <origin xyz="-0.02828 0.02828 0" rpy="0 0 0"/>
+            <origin xyz="0 0 0" rpy="0 0 0"/>
             <geometry>
                 <cylinder length="0.005" radius="0.01"/>
@@ -223,5 +234,5 @@
         <parent link="link1"/>
         <child link="hole4"/>
-        <origin xyz="0 0 0.01" rpy="0 0 0"/>
+        <origin xyz="-0.02828 0.02828 0.0125" rpy="0 0 0"/>
     </joint>
     <link name="hole5">
@@ -234,5 +245,5 @@
         </inertial>
         <visual>
-            <origin xyz="-0.04 0 0" rpy="0 0 0"/>
+            <origin xyz="0 0 0" rpy="0 0 0"/>
             <geometry>
                 <cylinder length="0.005" radius="0.01"/>
@@ -250,5 +261,5 @@
         <parent link="link1"/>
         <child link="hole5"/>
-        <origin xyz="0 0 0.01" rpy="0 0 0"/>
+        <origin xyz="-0.04 0 0.0125" rpy="0 0 0"/>
     </joint>
     <link name="hole6">
@@ -261,5 +272,5 @@
         </inertial>
         <visual>
-            <origin xyz="-0.02828 -0.02828 0" rpy="0 0 0"/>
+            <origin xyz="0 0 0" rpy="0 0 0"/>
             <geometry>
                 <cylinder length="0.005" radius="0.01"/>
@@ -277,5 +288,5 @@
         <parent link="link1"/>
         <child link="hole6"/>
-        <origin xyz="0 0 0.01" rpy="0 0 0"/>
+        <origin xyz="-0.02828 -0.02828 0.0125" rpy="0 0 0"/>
     </joint>
     <link name="hole7">
@@ -288,5 +299,5 @@
         </inertial>
         <visual>
-            <origin xyz="0 -0.04 0" rpy="0 0 0"/>
+            <origin xyz="0 0 0" rpy="0 0 0"/>
             <geometry>
                 <cylinder length="0.005" radius="0.01"/>
@@ -304,5 +315,5 @@
         <parent link="link1"/>
         <child link="hole7"/>
-        <origin xyz="0 0 0.01" rpy="0 0 0"/>
+        <origin xyz="0 -0.04 0.0125" rpy="0 0 0"/>
     </joint>
     <link name="hole8">
@@ -315,5 +326,5 @@
         </inertial>
         <visual>
-            <origin xyz="0.02828 -0.02828 0" rpy="0 0 0"/>
+            <origin xyz="0 0 0" rpy="0 0 0"/>
             <geometry>
                 <cylinder length="0.005" radius="0.01"/>
@@ -331,5 +342,5 @@
         <parent link="link1"/>
         <child link="hole8"/>
-        <origin xyz="0 0 0.01" rpy="0 0 0"/>
+        <origin xyz="0.02828 -0.02828 0.0125" rpy="0 0 0"/>
     </joint>
 </robot>

File: scara_v2_with_gripper/urdf/scara_and_rt_urdf.xacro (robot description, xacro)
@@ -152,4 +152,35 @@
         <axis xyz="1 0 0" />
     </joint>
+    <!--_______Colision object_______-->
+    <!--<link name="colisionBox">-->
+        <!--<inertial>-->
+            <!--<origin xyz="0 0 0" rpy="0 0 0" />-->
+            <!--<mass value="1" />-->
+            <!--<inertia ixx="1" ixy="0" ixz="0"-->
+                     <!--iyy="1" iyz="0"-->
+                     <!--izz="1" />-->
+        <!--</inertial>-->
+        <!--<visual>-->
+            <!--<origin xyz="0 0 0" rpy="0 0 0" />-->
+            <!--<geometry>-->
+                <!--<box size="0.05 0.05 0.2"/>-->
+            <!--</geometry>-->
+            <!--<material name="sensoSilver">-->
+            <!--</material>-->
+        <!--</visual>-->
+        <!--<collision>-->
+            <!--<origin xyz="0 0 0" rpy="0 0 0" />-->
+            <!--<geometry>-->
+                <!--<box size="0.1 0.1 0.2"/>-->
+            <!--</geometry>-->
+        <!--</collision>-->
+    <!--</link>-->
+    <!--<joint name="Joint_colisionBox" type="fixed">-->
+        <!--<parent link="BaseBox" />-->
+        <!--<child link="colisionBox" />-->
+        <!--<origin xyz="0.55 0.40 0.1" rpy="0 0 0" />-->
+        <!--<axis xyz="1 0 0" />-->
+    <!--</joint>-->
+    <!--**************************-->
     <link name="placeHole1">
         <inertial>
@@ -472,5 +503,5 @@
         </collision>
     </link>
-    <joint name="base_link1_to_link1" type="revolute">
+    <joint name="base_link1_to_link1" type="revolute"> <!-- rotary table joint-->
         <parent link="base_link1"/>
         <child link="link1"/>
@@ -786,18 +817,8 @@
         <axis xyz="0 1 0" />
         <!--<limit effort="0" lower="-2.65" upper="2.65" velocity="0"/>-->
-        <limit effort="0" lower="${-170*DEG2RAD}" upper="${170*DEG2RAD}" velocity="0"/>
+        <limit effort="0" lower="${-140*DEG2RAD}" upper="${140*DEG2RAD}" velocity="0"/>
     </joint>
     <!--**********************************-->
     <!--     GRIPPER JOINTS DEFINITION    -->
-    <!--     GRIPPER JOINTS DEFINITION    -->
-    <!--Revolute joint for IKfast-->
-    <!--<link name="fake_link"/>-->
-    <!--<joint name="fake_joint" type="revolute">-->
-        <!--<parent link="ScaraLink2" />-->
-        <!--<child link="fake_link" />-->
-        <!--<origin xyz="0 -0.0424 0.24305" rpy="1.57 0 3.1416" />-->
-        <!--<axis xyz="0 0 1" />-->
-        <!--<limit effort="1000.0" lower="0.0" upper="0.001" velocity="0"/>-->
-    <!--</joint>-->
     <link name="GripperBase">
         <inertial>

File: scara_v2_with_gripper/urdf/scara_v2_with_gripper_urdf.xacro (robot description, xacro)
@@ -155,5 +155,5 @@
     <link name="ScaraLink1">
         <inertial>
-            <origin xyz="0 0 0" rpy="-1.57 0 0" />
+            <origin xyz="0 0 0" rpy="0 0 0" />
             <mass value="3.8063" />
             <inertia ixx="7.8753E-3" ixy="4.6431E-3" ixz="-1.4702E-5"
@@ -162,5 +162,5 @@
         </inertial>
         <visual>
-            <origin xyz="0 0 0" rpy="-1.57 0 0" />
+            <origin xyz="0 0 0" rpy="0 0 0" />
             <geometry>
                 <mesh filename="package://scara_v2_with_gripper/meshes/ScaraLink1.STL" />   <!--ScaraLink1.STL-->
@@ -170,5 +170,5 @@
         </visual>
         <collision>
-            <origin xyz="0 0 0" rpy="-1.57 0 0" />
+            <origin xyz="0 0 0" rpy="0 0 0" />
             <geometry>
                 <mesh filename="package://scara_v2_with_gripper/meshes/ScaraLink1.STL" />
@@ -179,19 +179,19 @@
         <parent link="ScaraBase" />
         <child link="ScaraLink1" />
-        <origin xyz="0 0.051 0" rpy="1.57 0 0" />
-        <axis xyz="0 0 1" />
+        <origin xyz="0 0.051 0" rpy="0 0 0" />
+        <axis xyz="0 1 0" />
         <!--<limit effort="0" lower="-1.57079" upper="1.57079" velocity="0"/>-->
-        <limit effort="0" lower="${-85*DEG2RAD}" upper="${85*DEG2RAD}" velocity="0"/>
+        <limit effort="20" lower="${-85*DEG2RAD}" upper="${85*DEG2RAD}" velocity="100"/>        <!--100-->
     </joint>
     <link name="ScaraLink2">
         <inertial>
-            <origin xyz="0 0 0" rpy="1.57 1.57 0" />
+            <origin xyz="0 0 0" rpy="0 0 0" />
             <mass value="1.5020" />
             <inertia  ixx="5.0471E-2" ixy="3.0689E-4" ixz="-8.5622E-4"
-                    iyy="4.7456E-2" iyz="8.7643E-3"
-                    izz="5.2228E-3" />
-        </inertial>
-        <visual>
-            <origin  xyz="0 0 0" rpy="1.57 0 0" />
+                      iyy="4.7456E-2" iyz="8.7643E-3"
+                      izz="5.2228E-3" />
+        </inertial>
+        <visual>
+            <origin  xyz="0 0 0" rpy="0 0 0" />
             <geometry>
                 <mesh  filename="package://scara_v2_with_gripper/meshes/ScaraLink2.STL" />
@@ -201,5 +201,5 @@
         </visual>
         <collision>
-            <origin xyz="0 0 0" rpy="1.57 0 0" />
+            <origin xyz="0 0 0" rpy="0 0 0" />
             <geometry>
                 <mesh filename="package://scara_v2_with_gripper/meshes/ScaraLink2.STL" />
@@ -210,31 +210,21 @@
         <parent link="ScaraLink1" />
         <child link="ScaraLink2" />
-        <origin xyz="0.24972  0 0.081" rpy="0 0 1.57" />
-        <axis xyz="0 0 1" />
+        <origin xyz="0.24972 -0.081 0" rpy="3.14 -1.5708 0" />
+        <axis xyz="0 1 0" />
         <!--<limit effort="0" lower="-2.65" upper="2.65" velocity="0"/>-->
-        <limit effort="0" lower="${-170*DEG2RAD}" upper="${170*DEG2RAD}" velocity="0"/>
+        <limit effort="20" lower="${-170*DEG2RAD}" upper="${170*DEG2RAD}" velocity="100"/><!--100-->
     </joint>
     <!--**********************************-->
     <!--     GRIPPER JOINTS DEFINITION    -->
-    <!--Revolute joint for IKfast-->
-    <!--<link name="fake_link"/>-->
-    <!--<joint name="fake_joint" type="revolute">-->
-        <!--<parent link="ScaraLink2" />-->
-        <!--<child link="fake_link" />-->
-        <!--&lt;!&ndash;<origin xyz="0 -0.24305 0.0424 " rpy="0 0 3.1416" />&ndash;&gt;-->
-        <!--<origin xyz="0 -0.24305 -0.0424 " rpy="0 0 3.1416" />-->
-        <!--<axis xyz="0 0 1" />-->
-        <!--<limit effort="1000.0" lower="0.0" upper="0.001" velocity="0"/>-->
-    <!--</joint>-->
     <link name="GripperBase">
         <inertial>
-            <origin xyz="0 0 0" rpy="1.57 0 0" />
-            <mass  value="1" />
-            <inertia  ixx="1E-6" ixy="0" ixz="0"
-                    iyy="1E-6" iyz="0"
-                    izz="1E-6" />
-        </inertial>
-        <visual>
-            <origin  xyz="0 0 0"  rpy="1.57 0 0" />
+            <origin xyz="0 0 0" rpy="0 0 0" />
+            <mass  value="0.5" />
+            <inertia  ixx="0.01" ixy="0.01" ixz="0.01"
+                      iyy="0.01" iyz="0.01"
+                      izz="0.01" />
+        </inertial>
+        <visual>
+            <origin  xyz="0 0 0"  rpy="0 0 0" />
             <geometry>
                 <mesh filename="package://scara_v2_with_gripper/meshes/GripperBase.STL" />
@@ -244,5 +234,5 @@
         </visual>
         <collision>
-            <origin xyz="0 0 0" rpy="1.57 0 0" />
+            <origin xyz="0 0 0" rpy="0 0 0" />
             <geometry>
                 <mesh filename="package://scara_v2_with_gripper/meshes/GripperBase.STL" />
@@ -251,26 +241,23 @@
     </link>
     <joint name="Joint_GripperBase" type="prismatic">
-        <!--<parent link="fake_link" />-->
         <parent link="ScaraLink2" />
         <child link="GripperBase" />
-        <!--<origin xyz="0 0 0" rpy="0 0 0" />-->
-        <origin xyz="0 -0.24305 -0.0424 " rpy="0 0 3.1416" />
-        <axis xyz="0 0 1" />
-        <limit effort="1000.0" lower="-0.04" upper="0.05" velocity="1"/>
-    </joint>
-    <link name="tool0"/>
-    <joint name="Base_to_tool0" type="fixed">
-        <parent link="GripperBase" />
-        <child link="tool0" />
-        <origin xyz="0 0 0.0984" rpy="0 0 0 " />
-        <axis xyz="0 0 0" />
-    </joint>
+        <origin xyz="0 -0.0424 0.24305" rpy="3.1416 0 3.1416" />
+        <axis xyz="0 1 0" />
+        <limit effort="100.0" lower="-0.04" upper="0.05" velocity="1"/>
+    </joint>
+    <!--<joint name="Base_to_tool0" type="fixed">-->
+    <!--<parent link="GripperBase" />-->
+    <!--<child link="tool0" />-->
+    <!--<origin xyz="0 0.0984 0" rpy="0 0 0 " />-->
+    <!--</joint>-->
+    <!--<link name="tool0"/>-->
     <link name="GripperLeft">
         <inertial>
             <origin  xyz="0 0 0"  rpy="3.14 0 0" />
-            <mass value="1" />
-            <inertia ixx="1E-6"  ixy="0" ixz="0"
-                    iyy="1E-6" iyz="0"
-                    izz="1E-6" />
+            <mass value="0.1" />
+            <inertia  ixx="0.01" ixy="0.01" ixz="0.01"
+                      iyy="0.01" iyz="0.01"
+                      izz="0.01" />
         </inertial>
         <visual>
@@ -292,15 +279,15 @@
         <parent link="GripperBase" />
         <child link="GripperLeft" />
-        <origin xyz="-0.0162 0 0.0984" rpy="-1.57 0 0" />
+        <origin xyz="-0.0162 0.0984 0" rpy="3.1416 0 0" />
         <axis xyz="1 0 0" />
-        <limit effort="1000.0" lower="0" upper="0.003" velocity="1"/>
+        <limit effort="100.0" lower="0" upper="0.003" velocity="1"/>
     </joint>
     <link name="GripperRight">
         <inertial>
             <origin   xyz="0 0 0" rpy="3.14 0 0" />
-            <mass value="1" />
-            <inertia  ixx="1E-6"  ixy="0" ixz="0"
-                    iyy="1E-6" iyz="0"
-                    izz="1E-6" />
+            <mass value="0.1" />
+            <inertia  ixx="0.01" ixy="0.01" ixz="0.01"
+                      iyy="0.01" iyz="0.01"
+                      izz="0.01" />
         </inertial>
         <visual>
@@ -322,5 +309,5 @@
         <parent link="GripperBase" />
         <child link="GripperRight" />
-        <origin  xyz="0.0165 0 0.0984" rpy="1.57 0 3.1416" />
+        <origin  xyz="0.0165 0.0984 0" rpy="3.1416 0 3.1416" />
         <axis  xyz="1 0 0" />
         <limit effort="1000.0" lower="0" upper="0.003" velocity="1"/>
