Commit message: Modified RT  control in scara_v2_full_controll
TO DO: modify  connect moveit and gazebo of RT, find out how to add RT to SCARA moveit.

Signed-off-by: senso-viktor <viktordluhos@gmail.com>

File: gazebo_scara_and_rt/scara_v2_full_description/urdf/rotary_table_v3_urdf.xacro (robot description, xacro)
@@ -227,3 +227,15 @@
         <axis xyz="0 0 0" />
     </joint>
+    <!--***************** Transmision definitions *******************************-->
+    <transmission name="tran1rt">
+        <type>transmission_interface/SimpleTransmission</type>
+        <joint name="rotary_table_joint">
+            <hardwareInterface>EffortJointInterface</hardwareInterface>
+        </joint>
+        <actuator name="motor1">
+            <hardwareInterface>EffortJointInterface</hardwareInterface>
+            <mechanicalReduction>1</mechanicalReduction>
+        </actuator>
+    </transmission>
+    <!--*************************************************************************-->
 </robot>
